File: vca_lm13700.kicad_sch (KiCad schematic)
At the start: 20 parts, among them Q201 Q_PNP_BEC, U201 LM13700, U202 MCP6004, U203 MCP6004

Commit message: VCF layout
Parts:
- removed U202, U203: MCP6004, Package_SO:SOIC-14_3.9x8.7mm_P1.27mm, symbol Amplifier_Operational:MCP6004
- added C202, C203, C204, C206, C207, C208: 100n, Capacitor_SMD:C_0603_1608Metric_Pad1.08x0.95mm_HandSolder, symbol Device:C
- added C205: 100p, Capacitor_SMD:C_0603_1608Metric_Pad1.08x0.95mm_HandSolder, symbol Device:C
- added Q202: Q_PNP_BEC, Package_TO_SOT_SMD:SOT-23_Handsoldering, symbol Device:Q_PNP_BEC
- added R213, R214, R218, R224: 200K, Resistor_SMD:R_0603_1608Metric_Pad0.98x0.95mm_HandSolder, symbol Device:R
- added R215: 1M, Resistor_SMD:R_0603_1608Metric_Pad0.98x0.95mm_HandSolder, symbol Device:R
- added R216, R217: 100K, Resistor_SMD:R_0603_1608Metric_Pad0.98x0.95mm_HandSolder, symbol Device:R
- added R219: 10K, Resistor_SMD:R_0603_1608Metric_Pad0.98x0.95mm_HandSolder, symbol Device:R
- added R220: 1K, Resistor_SMD:R_0603_1608Metric_Pad0.98x0.95mm_HandSolder, symbol Device:R
- added R221: 680, Resistor_SMD:R_0603_1608Metric_Pad0.98x0.95mm_HandSolder, symbol Device:R
- added R222: 30K, Resistor_SMD:R_0603_1608Metric_Pad0.98x0.95mm_HandSolder, symbol Device:R
- added R223: 5K, Resistor_SMD:R_0603_1608Metric_Pad0.98x0.95mm_HandSolder, symbol Device:R
- added RV204: 100K, Potentiometer_SMD:Potentiometer_Bourns_3314J_Vertical, symbol Device:R_Potentiometer_Trim
- added U202: MCP6002, symbol Amplifier_Operational:MCP6002-xSN
- added U203: TL072, symbol Amplifier_Operational:TL072
- C201: value 470p -> 100p
- R212: value 20K -> 1M
- RV201: value 100K multiturn -> 100K
Connections:
- net +4.5V: now also R213.1, R218.1, R221.2, R222.2, U202.3 (+), U202.5 (+)
- net +9V: now also U201.11 (V+), C206.1, C207.1, RV204.1, U202.8 (V+), U203.8 (V+)
- net GND: now also R212.2, U201.6 (V-), C206.2, C207.2, R214.2, R215.2, R223.2, R224.2, RV204.3, U202.4 (V-), U203.4 (V-)
- net at C201.1, R203.2, R204.2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: now also U202.2 (-)
- net at U201.5: now also U201.7, R222.1; no longer R212.1
- net at R210.1: now also U203.6 (-), U203.7
- net at R208.1, U201.9: now also C203.1
- net at Q201.1 (B): now also U202.1
- net VCA2_Iabc: now reaches U201.1
- net VCA2_Iabc: now also R220.1
- net at U201.8: now also C208.1, R223.1
- net A1_IN: no longer names the net of R201.1
- net A1_IN: now also U203.1, U203.2 (-)
- net CV1_IN renamed VCA1_CV
- net Iabc1 renamed VCA1_Iabc
- new net: R216.1, RV204.2
- new net: C205.1, R216.2, R217.2, R219.1, U202.6 (-)
- new net: Q202.1 (B), U202.7
- new net: C204.2, R218.2, U203.5 (+)
- new net: C205.2, Q202.2 (E), R219.2, R221.1
- new net: Q202.3 (C), R220.2
- new net: C202.2, R213.2, U203.3 (+)
- new net VCA1_In: C202.1, R212.1
- new net VCA1_Out: C203.2, R214.1
- new net VCA2_CV: R217.1
- new net VCA2_In: C204.1, R215.1
- new net VCA2_Out: C208.2, R224.1
Other:
- added sheet Audio VCA IO (audio-vca-io.kicad_sch)
- note added: "Audio VCA"
- note removed: "CV biased to 4.5V as input Gives 2V-6.8V range on the output with the VCA fully on 4.9V at the output with the VCA fully off Iabc circuit is the same as for audio"
- note removed: "Cap sets the LPF cutoff at 34kHz"
- note removed: "TODO: check pinout of transistor with the footprint"
- moved on the sheet: C201, Q201, R201, R202, R203, R204, R205, R206, R207, R208, R209, R210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
