File: vcf.kicad_sch (KiCad schematic)
At the start: 57 parts, among them U601 TL074, U602 TL074, U603 SSI2164

Commit message: VCF layout
Parts:
- removed C609, C611: 100n, Capacitor_SMD:C_0603_1608Metric_Pad1.08x0.95mm_HandSolder, symbol Device:C
- added D606: D_TVS, Diode_SMD:D_SOD-323_HandSoldering, symbol Device:D_TVS
- added H602: In, MountingHole:MountingHole_4.3mm_M4_Pad_TopBottom, symbol Mechanical:MountingHole_Pad
Connections:
- net +4.5V: now also U602.10 (+), U602.12 (+), U602.3 (+), U602.5 (+); no longer U602.10 (+), U602.12 (+), U602.3 (+), U602.5 (+)
- net GND: now also D606.1 (A1)
- net HP: now also U602.14; no longer U602.1
- net In: now also D606.2 (A2), H602.1
- net LBP: now also U602.7; no longer U602.8
- net LP: now also U602.1; no longer U602.14
- net UBP: now also U602.8; no longer U602.7
- net VCA_I_In1: now also R612.2, R614.1; no longer R613.2, R619.1
- net VCA_I_In2: now also R630.2, R631.1; no longer R626.2, R629.1
- net VCA_I_In3: now also R626.2, R629.1; no longer R630.2, R631.1
- net VCA_I_In4: now also R613.2, R619.1; no longer R612.2, R614.1
- net VCA_I_Out1: now also R623.2, R624.1, R625.2, R627.1, U601.6 (-); no longer C605.1, U602.6 (-)
- net VCA_I_Out2: now also C614.1, U602.2 (-); no longer C608.1, U602.9 (-)
- net VCA_I_Out3: now also C608.1, U602.6 (-); no longer C614.1, U602.13 (-)
- net VCA_I_Out4: now also C605.1, U602.9 (-); no longer R623.2, R624.1, R625.2, R627.1, U601.6 (-)
- net at R609.2, R610.2, R611.1: now also U602.13 (-); no longer U602.2 (-)
Other:
- moved on the sheet: D603, H601
