File: vcf.kicad_sch (KiCad schematic)
At the start: 80 parts

Commit message: VCF schem combed
Parts:
- removed C?: 100n, symbol Device:C
- removed R? (x8): 100K, symbol Device:R
- removed R? (x5): 10K, symbol Device:R
- removed R?: 200K, symbol Device:R
- removed R?: 1K, symbol Device:R
- removed RV? (x4): B100K, R0904NB10KL-25KQ:V2_TRIM_R0904NB10KL-25KQ-, symbol R0904NB10KL-25KQ:R_Potentiometer_Shield
- removed U? (x6): TL074, symbol Amplifier_Operational:TL074
- added C606: 100n, Capacitor_SMD:C_0603_1608Metric_Pad1.08x0.95mm_HandSolder, symbol Device:C
- added D603: D_TVS, Diode_SMD:D_SOD-323_HandSoldering, symbol Device:D_TVS
- added H601: Main_Out, MountingHole:MountingHole_4.3mm_M4_Pad_TopBottom, symbol Mechanical:MountingHole_Pad
- added R615, R616, R617, R618, R620: 10K, Resistor_SMD:R_0603_1608Metric_Pad0.98x0.95mm_HandSolder, symbol Device:R
- added R622: 1K, Resistor_SMD:R_0603_1608Metric_Pad0.98x0.95mm_HandSolder, symbol Device:R
- added R628: 200K, Resistor_SMD:R_0603_1608Metric_Pad0.98x0.95mm_HandSolder, symbol Device:R
- added unit 4 of U601
- C601, C602, C603, C604, C605, C607, C608, C609, C610, C611, C612, C613, C614, C615, C616: renamed from C?; footprint (none) -> Capacitor_SMD:C_0603_1608Metric_Pad1.08x0.95mm_HandSolder
- D601, D602: renamed from D?; footprint (none) -> Diode_SMD:D_SOD-323_HandSoldering
- D604, D605: renamed from D?; footprint (none) -> Diode_SMD:D_SOD-123
- R601, R602, R603, R604, R605, R606, R607, R608, R609, R610, R611, R612, R613, R614, R619, R621, R623, R624, R625, R626, R627, R629, R630, R631, R632: renamed from R?; footprint (none) -> Resistor_SMD:R_0603_1608Metric_Pad0.98x0.95mm_HandSolder
- U601, U602: renamed from U?; footprint (none) -> Package_SO:SOIC-14_3.9x8.7mm_P1.27mm
- gave numbers to parts that had none: 1
Connections:
- net +4.5V: now also U601.12 (+)
- net GND: now also D603.1 (A1), R628.2
- net HP_Vert: now also R615.1
- net LBP_Vert: now also R617.1
- net LP_Vert: now also R618.1
- net Out: now also C606.2, D603.2 (A2), H601.1, R628.1
- net UBP_Vert: now also R616.1
- new net: R615.2, R616.2, R617.2, R618.2, R620.1, U601.13 (-)
- new net: R620.2, R622.1, U601.14
- new net: C606.1, R622.2
Other:
- sheet VCF Audio Outs ports: added +4.5V, +9V, GND, HP_In, HP_Vert, LBP_In, LBP_Vert, LP_In, LP_Vert, UBP_In, UBP_Vert; removed none
- moved on the sheet: C609, C611, C612, C613, U601E, U602E

Commit message: Start VCF layout
Parts:
- removed C609, C611: 100n, Capacitor_SMD:C_0603_1608Metric_Pad1.08x0.95mm_HandSolder, symbol Device:C
- added D606: D_TVS, Diode_SMD:D_SOD-323_HandSoldering, symbol Device:D_TVS
- added H602: In, MountingHole:MountingHole_4.3mm_M4_Pad_TopBottom, symbol Mechanical:MountingHole_Pad
Connections:
- net GND: now also D606.1 (A1)
- net In: now also D606.2 (A2), H602.1
Other:
- moved on the sheet: D603, H601

Commit message: WIP VCF Layout
Connections:
- net +4.5V: now also U602.10 (+), U602.12 (+), U602.3 (+), U602.5 (+); no longer U602.10 (+), U602.12 (+), U602.3 (+), U602.5 (+)
- net HP: now also U602.14; no longer U602.1
- net LBP: now also U602.7; no longer U602.8
- net LP: now also U602.1; no longer U602.14
- net UBP: now also U602.8; no longer U602.7
- net VCA_I_In1: now also R612.2, R614.1; no longer R613.2, R619.1
- net VCA_I_In2: now also R630.2, R631.1; no longer R626.2, R629.1
- net VCA_I_In3: now also R626.2, R629.1; no longer R630.2, R631.1
- net VCA_I_In4: now also R613.2, R619.1; no longer R612.2, R614.1
- net VCA_I_Out1: now also R623.2, R624.1, R625.2, R627.1, U601.6 (-); no longer C605.1, U602.6 (-)
- net VCA_I_Out2: now also C614.1, U602.2 (-); no longer C608.1, U602.9 (-)
- net VCA_I_Out3: now also C608.1, U602.6 (-); no longer C614.1, U602.13 (-)
- net VCA_I_Out4: now also C605.1, U602.9 (-); no longer R623.2, R624.1, R625.2, R627.1, U601.6 (-)
- net at R609.2, R610.2, R611.1: now also U602.13 (-); no longer U602.2 (-)
Changed lines of the file:
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@@
     (effects (font (size 1.27 1.27)) (justify left bottom))
   )
-  (label "VCA_I_In4" (at 101.6 97.79 0)
+  (label "VCA_I_In4" (at 107.95 39.37 0)
     (effects (font (size 1.27 1.27)) (justify left bottom))
   )
@@
     (effects (font (size 1.27 1.27)) (justify left bottom))
   )
-  (label "VCA_I_Out4" (at 137.16 109.22 180)
+  (label "VCA_I_Out4" (at 129.54 39.37 180)
     (effects (font (size 1.27 1.27)) (justify right bottom))
   )
@@
     (effects (font (size 1.27 1.27)) (justify right bottom))
   )
-  (label "VCA_I_Out1" (at 129.54 39.37 180)
+  (label "VCA_I_Out1" (at 137.16 109.22 180)
     (effects (font (size 1.27 1.27)) (justify right bottom))
   )
@@
     (effects (font (size 1.27 1.27)) (justify right bottom))
   )
-  (label "VCA_I_In2" (at 165.1 41.91 0)
+  (label "VCA_I_In2" (at 227.33 41.91 0)
     (effects (font (size 1.27 1.27)) (justify left bottom))
   )
@@
     (effects (font (size 1.27 1.27)) (justify right bottom))
   )
-  (label "VCA_I_In1" (at 107.95 39.37 0)
+  (label "VCA_I_In1" (at 101.6 97.79 0)
     (effects (font (size 1.27 1.27)) (justify left bottom))
   )
@@
     (effects (font (size 1.27 1.27)) (justify left bottom))
   )
-  (label "VCA_I_Out2" (at 187.96 39.37 180)
-    (effects (font (size 1.27 1.27)) (justify right bottom))
-  )
-  (label "VCA_I_In3" (at 227.33 41.91 0)
+  (label "VCA_I_Out2" (at 248.92 39.37 180)
+    (effects (font (size 1.27 1.27)) (justify right bottom))
+  )
+  (label "VCA_I_In3" (at 165.1 41.91 0)
     (effects (font (size 1.27 1.27)) (justify left bottom))
   )
@@
     (effects (font (size 1.27 1.27)) (justify right bottom))
   )
-  (label "VCA_I_Out3" (at 248.92 39.37 180)
+  (label "VCA_I_Out3" (at 187.96 39.37 180)
     (effects (font (size 1.27 1.27)) (justify right bottom))
   )
@@
     (effects (font (size 1.27 1.27)) (justify right))
   )
-  (symbol (lib_id "Amplifier_Operational:TL074") (at 140.97 41.91 0) (mirror x) (unit 2)
+  (symbol (lib_id "Amplifier_Operational:TL074") (at 140.97 41.91 0) (mirror x) (unit 3)
     (in_bom yes) (on_board yes) (fields_autoplaced)
     (property "Reference" "U602" (id 0) (at 140.97 31.75 0))
@@
     (pin "1")
   )
-  (symbol (lib_id "Amplifier_Operational:TL074") (at 261.62 41.91 0) (mirror x) (unit 4)
+  (symbol (lib_id "Amplifier_Operational:TL074") (at 261.62 41.91 0) (mirror x) (unit 1)
     (in_bom yes) (on_board yes) (fields_autoplaced)
     (property "Reference" "U602" (id 0) (at 261.62 31.75 0))
@@
     (pin "2")
   )
-  (symbol (lib_id "Amplifier_Operational:TL074") (at 200.66 41.91 0) (mirror x) (unit 3)
+  (symbol (lib_id "Amplifier_Operational:TL074") (at 200.66 41.91 0) (mirror x) (unit 2)
     (in_bom yes) (on_board yes) (fields_autoplaced)
     (property "Reference" "U602" (id 0) (at 200.66 31.75 0))
@@
     (pin "2")
   )
-  (symbol (lib_id "Amplifier_Operational:TL074") (at 83.82 39.37 0) (mirror x) (unit 1)
+  (symbol (lib_id "Amplifier_Operational:TL074") (at 83.82 39.37 0) (mirror x) (unit 4)
     (in_bom yes) (on_board yes) (fields_autoplaced)
     (property "Reference" "U602" (id 0) (at 83.82 29.21 0))
