File: vcf.kicad_sch (KiCad schematic)
At the start: 57 parts, among them U601 TL074, U602 TL074, U603 SSI2164

Commit message: Increase the size of dc blocking caps
Parts:
- C601, C606: value 100n -> 470n; footprint Capacitor_SMD:C_0603_1608Metric_Pad1.08x0.95mm_HandSolder -> Capacitor_SMD:C_0805_2012Metric_Pad1.18x1.45mm_HandSolder
Changed lines of the file:
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@@
+    (pin "2")
+  )
+  (symbol (lib_id "Device:C") (at 149.86 148.59 90) (unit 1)
+    (in_bom yes) (on_board yes) (fields_autoplaced)
+    (property "Reference" "C606" (id 0) (at 149.86 140.97 90))
+    (property "Value" "470n" (id 1) (at 149.86 143.51 90))
+    (property "Footprint" "Capacitor_SMD:C_0805_2012Metric_Pad1.18x1.45mm_HandSolder" (id 2) (at 153.67 147.6248 0)
+      (effects (font (size 1.27 1.27)) hide)
+    )
+    (property "Datasheet" "~" (id 3) (at 149.86 148.59 0)
+      (effects (font (size 1.27 1.27)) hide)
+    )
+    (pin "1")
     (pin "2")
   )
@@
     (pin "2")
   )
-  (symbol (lib_id "Device:C") (at 149.86 148.59 90) (unit 1)
-    (in_bom yes) (on_board yes) (fields_autoplaced)
-    (property "Reference" "C606" (id 0) (at 149.86 140.97 90))
-    (property "Value" "100n" (id 1) (at 149.86 143.51 90))
-    (property "Footprint" "Capacitor_SMD:C_0603_1608Metric_Pad1.08x0.95mm_HandSolder" (id 2) (at 153.67 147.6248 0)
-      (effects (font (size 1.27 1.27)) hide)
-    )
-    (property "Datasheet" "~" (id 3) (at 149.86 148.59 0)
-      (effects (font (size 1.27 1.27)) hide)
-    )
-    (pin "1")
-    (pin "2")
-  )
-  (symbol (lib_id "Device:C") (at 33.02 39.37 90) (unit 1)
-    (in_bom yes) (on_board yes) (fields_autoplaced)
-    (property "Reference" "C601" (id 0) (at 33.02 31.75 90))
-    (property "Value" "100n" (id 1) (at 33.02 34.29 90))
-    (property "Footprint" "Capacitor_SMD:C_0603_1608Metric_Pad1.08x0.95mm_HandSolder" (id 2) (at 36.83 38.4048 0)
-      (effects (font (size 1.27 1.27)) hide)
-    )
-    (property "Datasheet" "~" (id 3) (at 33.02 39.37 0)
-      (effects (font (size 1.27 1.27)) hide)
-    )
-    (pin "1")
-    (pin "2")
-  )
   (symbol (lib_id "Device:R") (at 22.86 43.18 0) (unit 1)
     (in_bom yes) (on_board yes) (fields_autoplaced)
@@
       (effects (font (size 1.27 1.27)) hide)
     )
+    (pin "1")
+    (pin "2")
+  )
+  (symbol (lib_id "Device:C") (at 33.02 39.37 90) (unit 1)
+    (in_bom yes) (on_board yes) (fields_autoplaced)
+    (property "Reference" "C601" (id 0) (at 33.02 31.75 90))
+    (property "Value" "470n" (id 1) (at 33.02 34.29 90))
+    (property "Footprint" "Capacitor_SMD:C_0805_2012Metric_Pad1.18x1.45mm_HandSolder" (id 2) (at 36.83 38.4048 0)
+      (effects (font (size 1.27 1.27)) hide)
+    )
+    (property "Datasheet" "~" (id 3) (at 33.02 39.37 0)
+      (effects (font (size 1.27 1.27)) hide)
+    )

Commit message: Add JLC parts numbers
Parts:
- C601, C606: LCSC (none) -> C651004; Role (none) -> audio-coupling
- C602, C605, C608, C614: LCSC (none) -> C307359; Role (none) -> audio-filter
- C603, C604, C607, C610: LCSC (none) -> C342931; Role (none) -> audio-filter
- C612, C613, C615, C616: LCSC (none) -> C497032; Role (none) -> ic-bypass
- D601, D602: value D -> 1N4148; LCSC (none) -> C2128
- D603, D606: LCSC (none) -> C20936
- D604, D605: value D_Zener -> 2.1V Zener; LCSC (none) -> C2992021
- R601: LCSC (none) -> C234360
- R602, R603, R604, R605, R607, R608, R609, R610, R611, R613, R623, R625, R626, R630: LCSC (none) -> C138282
- R606, R628: LCSC (none) -> C203392
- R612: LCSC (none) -> C2907015
- R614, R619, R629, R631: LCSC (none) -> C203410
- R615, R616, R617, R618, R620: LCSC (none) -> C98220
- R621, R632: LCSC (none) -> C144661
- R622: LCSC (none) -> C2907002
- R624: LCSC (none) -> C328354
- R627: LCSC (none) -> C2907025
- U601, U602: LCSC (none) -> C6963
