File: konstrukt-kicad6.kicad_pcb (KiCad board)
At the start: 2 copper layers, 87.5 x 172.1 mm, 147 parts, among them Q201 Q_PNP_BEC, U201 LM13700, U202 MCP6004, U203 MCP6004, U301 MCP6004, U302 TL072, U401 MCP6004, U402 TL072, U501 MCP6004, U502 TL072

Commit message: Moved design to the PCB
Parts:
- removed the ? at (106.4, 16.4)
- removed C401, C402, C403, C404, C501, C502, C503, C504: 30p, Capacitor_SMD:C_0603_1608Metric_Pad1.08x0.95mm_HandSolder
- removed C405, C406, C505, C506: 100n, Capacitor_SMD:C_0603_1608Metric_Pad1.08x0.95mm_HandSolder
- removed D401, D402, D403, D404, D501, D502, D503, D504: D_TVS, Diode_SMD:D_SOD-323_HandSoldering
- removed D405, D406, D505, D506: LED_Green, LED_THT:LED_D3.0mm
- removed D407, D408, D507, D508: LED_Yellow, LED_THT:LED_D3.0mm
- removed H401: 2xAttenuverters2_1_In, MountingHole:MountingHole_4.3mm_M4_Pad_TopBottom
- removed H402: 2xAttenuverters2_1_Out, MountingHole:MountingHole_4.3mm_M4_Pad_TopBottom
- removed H403: 2xAttenuverters2_2_In, MountingHole:MountingHole_4.3mm_M4_Pad_TopBottom
- removed H404: 2xAttenuverters2_2_Out, MountingHole:MountingHole_4.3mm_M4_Pad_TopBottom
- removed H501: 2xAttenuverters3_1_In, MountingHole:MountingHole_4.3mm_M4_Pad_TopBottom
- removed H502: 2xAttenuverters3_1_Out, MountingHole:MountingHole_4.3mm_M4_Pad_TopBottom
- removed H503: 2xAttenuverters3_2_In, MountingHole:MountingHole_4.3mm_M4_Pad_TopBottom
- removed H504: 2xAttenuverters3_2_Out, MountingHole:MountingHole_4.3mm_M4_Pad_TopBottom
- removed R401, R402, R403, R404, R405, R406, R407, R408, R409, R410, R414, R416, R501, R502, R503, R504, R505, R506, R507, R508, R509, R510, R514, R516: 100K, Resistor_SMD:R_0603_1608Metric_Pad0.98x0.95mm_HandSolder
- removed R411, R412, R511, R512: 1K, Resistor_SMD:R_0603_1608Metric_Pad0.98x0.95mm_HandSolder
- removed R413, R415, R513, R515: 470, Resistor_SMD:R_0603_1608Metric_Pad0.98x0.95mm_HandSolder
- removed R417, R418, R517, R518: 20K, Resistor_SMD:R_0603_1608Metric_Pad0.98x0.95mm_HandSolder
- removed RV401, RV402, RV403, RV404, RV501, RV502, RV503, RV504: B100K, R0904NB10KL-25KQ:V2_TRIM_R0904NB10KL-25KQ-
- removed U401, U501: MCP6004, Package_SO:TSSOP-14_4.4x5mm_P0.65mm
- removed U402, U502: TL072, Package_SO:SOIC-8_3.9x4.9mm_P1.27mm
- added ? (x3): , Graphics, B.Cu at (378.4, 21.7)
- moved R202 349.4 mm to (318.5, -75.8)
- moved R207 349.4 mm to (326.3, -83.9)
- moved R211 349.4 mm to (318.5, -73.3)
- moved R212 349.4 mm to (330.8, -90.9)
- moved RV201 349.4 mm to (316.7, -80.9)
- moved U202 349.4 mm to (311.7, -88.9)
- moved U203 349.4 mm to (303.3, -77.5)
- moved C201 349.4 mm to (324.3, -86.4)
- moved Q201 349.4 mm to (325.4, -89.9)
- moved R201 349.4 mm to (314.2, -73.3)
- moved R203 349.4 mm to (309.8, -76.8)
- moved R204 349.4 mm to (314.2, -75.8)
- moved R205 349.4 mm to (321.9, -80.9)
- moved R206 349.4 mm to (321.9, -83.4)
- moved R208 349.4 mm to (328.7, -86.4)
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Routing:
- net /+9V: track 603.7 -> 131.2 mm, vias 21 -> 6
- net /+4.5V: track 525.0 -> 188.4 mm, vias 42 -> 14
- net Net-(C503-Pad2): track 133.2 -> 0.00 mm, vias 2 -> 0
- net Net-(C403-Pad2): track 133.2 -> 0.00 mm, vias 2 -> 0
- net Net-(C504-Pad2): track 125.4 -> 0.00 mm, vias 6 -> 0
- net Net-(C404-Pad2): track 125.4 -> 0.00 mm, vias 6 -> 0
- net Net-(R405-Pad2): track 62.5 -> 0.00 mm
- net Net-(R505-Pad2): track 62.5 -> 0.00 mm
- net Net-(RV401-Pad2): track 59.9 -> 0.00 mm
- net Net-(RV501-Pad2): track 59.9 -> 0.00 mm
- net /2xAttenuverters3/2xAttenuverters2_1_In: track 54.4 -> 0.00 mm
- net /2xAttenuverters2/2xAttenuverters2_1_In: track 54.4 -> 0.00 mm
- net /2xAttenuverters3/2xAttenuverters2_2_In: track 53.6 -> 0.00 mm, vias 2 -> 0
- net /2xAttenuverters2/2xAttenuverters2_2_In: track 53.6 -> 0.00 mm, vias 2 -> 0
- net Net-(C503-Pad1): track 44.5 -> 0.00 mm, vias 2 -> 0
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Other:
- board size 87.5 x 172.1 mm -> 356.9 x 210 mm

Commit message: Attenuverters laid out
Parts:
- removed C201: small??, Capacitor_SMD:C_0603_1608Metric_Pad1.08x0.95mm_HandSolder
- removed Q201: Q_PNP_BEC, Package_TO_SOT_SMD:SOT-23_Handsoldering
- removed R201, R206, R210: 30K, Resistor_SMD:R_0603_1608Metric_Pad0.98x0.95mm_HandSolder
- removed R202, R211: 8.2K, Resistor_SMD:R_0603_1608Metric_Pad0.98x0.95mm_HandSolder
- removed R203, R204: 100K, Resistor_SMD:R_0603_1608Metric_Pad0.98x0.95mm_HandSolder
- removed R205: 10K, Resistor_SMD:R_0603_1608Metric_Pad0.98x0.95mm_HandSolder
- removed R207: 1K, Resistor_SMD:R_0603_1608Metric_Pad0.98x0.95mm_HandSolder
- removed R208: 5K, Resistor_SMD:R_0603_1608Metric_Pad0.98x0.95mm_HandSolder
- removed R209: 680, Resistor_SMD:R_0603_1608Metric_Pad0.98x0.95mm_HandSolder
- removed R212: 20K, Resistor_SMD:R_0603_1608Metric_Pad0.98x0.95mm_HandSolder
- removed RV201: 100K multiturn, Potentiometer_SMD:Potentiometer_Bourns_3314J_Vertical
- removed RV202, RV203: 1K, Potentiometer_SMD:Potentiometer_Bourns_3314J_Vertical
- removed U201: LM13700, Package_SO:SOIC-16_3.9x9.9mm_P1.27mm
- removed U202, U203: MCP6004, Package_SO:TSSOP-14_4.4x5mm_P0.65mm
- added C401: 30p, Capacitor_SMD:C_0603_1608Metric_Pad1.08x0.95mm_HandSolder, F.Cu at (138.0, 143.7)
- added C402: 30p, Capacitor_SMD:C_0603_1608Metric_Pad1.08x0.95mm_HandSolder, F.Cu at (154.7, 153.0)
- added C403: 30p, Capacitor_SMD:C_0603_1608Metric_Pad1.08x0.95mm_HandSolder, F.Cu at (131.6, 143.7)
- added C404: 30p, Capacitor_SMD:C_0603_1608Metric_Pad1.08x0.95mm_HandSolder, F.Cu at (186.9, 143.7)
- added C405: 100n, Capacitor_SMD:C_0603_1608Metric_Pad1.08x0.95mm_HandSolder, F.Cu at (149.0, 148.0)
- added C406: 100n, Capacitor_SMD:C_0603_1608Metric_Pad1.08x0.95mm_HandSolder, F.Cu at (161.1, 159.2)
- added C501: 30p, Capacitor_SMD:C_0603_1608Metric_Pad1.08x0.95mm_HandSolder, F.Cu at (138.0, 187.8)
- added C502: 30p, Capacitor_SMD:C_0603_1608Metric_Pad1.08x0.95mm_HandSolder, F.Cu at (154.7, 197.1)
- added C503: 30p, Capacitor_SMD:C_0603_1608Metric_Pad1.08x0.95mm_HandSolder, F.Cu at (131.6, 187.8)
- added C504: 30p, Capacitor_SMD:C_0603_1608Metric_Pad1.08x0.95mm_HandSolder, F.Cu at (186.9, 187.8)
- added C505: 100n, Capacitor_SMD:C_0603_1608Metric_Pad1.08x0.95mm_HandSolder, F.Cu at (149.0, 192.1)
- added C506: 100n, Capacitor_SMD:C_0603_1608Metric_Pad1.08x0.95mm_HandSolder, F.Cu at (161.1, 203.3)
- added D401: D_TVS, Diode_SMD:D_SOD-323_HandSoldering, F.Cu at (125.5, 156.5)
- added D402: D_TVS, Diode_SMD:D_SOD-323_HandSoldering, F.Cu at (137.0, 160.3)
- added D403: D_TVS, Diode_SMD:D_SOD-323_HandSoldering, F.Cu at (167.4, 155.9)
- added D404: D_TVS, Diode_SMD:D_SOD-323_HandSoldering, F.Cu at (184.6, 161.6)
- added D405: LED_Green, LED_THT:LED_D3.0mm, B.Cu at (133.0, 148.5)
- added D406: LED_Green, LED_THT:LED_D3.0mm, B.Cu at (174.5, 148.5)
- added D407: LED_Yellow, LED_THT:LED_D3.0mm, B.Cu at (133.0, 154.5)
- added D408: LED_Yellow, LED_THT:LED_D3.0mm, B.Cu at (174.5, 154.5)
- added D501: D_TVS, Diode_SMD:D_SOD-323_HandSoldering, F.Cu at (125.5, 200.6)
- added D502: D_TVS, Diode_SMD:D_SOD-323_HandSoldering, F.Cu at (137.0, 204.4)
- added D503: D_TVS, Diode_SMD:D_SOD-323_HandSoldering, F.Cu at (167.4, 200.0)
- added D504: D_TVS, Diode_SMD:D_SOD-323_HandSoldering, F.Cu at (184.6, 205.7)
- added D505: LED_Green, LED_THT:LED_D3.0mm, B.Cu at (133.0, 192.6)
- added D506: LED_Green, LED_THT:LED_D3.0mm, B.Cu at (174.5, 192.6)
- added D507: LED_Yellow, LED_THT:LED_D3.0mm, B.Cu at (133.0, 198.6)
- added D508: LED_Yellow, LED_THT:LED_D3.0mm, B.Cu at (174.5, 198.6)
- added H401: 2xAttenuverters2_1_In, MountingHole:MountingHole_4.3mm_M4_Pad_TopBottom, B.Cu at (125.6, 148.5)
- added H402: 2xAttenuverters2_1_Out, MountingHole:MountingHole_4.3mm_M4_Pad_TopBottom, B.Cu at (142.9, 154.5)
- added H403: 2xAttenuverters2_2_In, MountingHole:MountingHole_4.3mm_M4_Pad_TopBottom, B.Cu at (167.2, 148.5)
- added H404: 2xAttenuverters2_2_Out, MountingHole:MountingHole_4.3mm_M4_Pad_TopBottom, B.Cu at (184.5, 154.5)
- added H501: 2xAttenuverters3_1_In, MountingHole:MountingHole_4.3mm_M4_Pad_TopBottom, B.Cu at (125.6, 192.6)
- added H502: 2xAttenuverters3_1_Out, MountingHole:MountingHole_4.3mm_M4_Pad_TopBottom, B.Cu at (142.9, 198.6)
- added H503: 2xAttenuverters3_2_In, MountingHole:MountingHole_4.3mm_M4_Pad_TopBottom, B.Cu at (167.2, 192.6)
- added H504: 2xAttenuverters3_2_Out, MountingHole:MountingHole_4.3mm_M4_Pad_TopBottom, B.Cu at (184.5, 198.6)
- added R401: 100K, Resistor_SMD:R_0603_1608Metric_Pad0.98x0.95mm_HandSolder, F.Cu at (149.0, 143.7)
- added R402: 100K, Resistor_SMD:R_0603_1608Metric_Pad0.98x0.95mm_HandSolder, F.Cu at (161.1, 148.7)
- added R403: 100K, Resistor_SMD:R_0603_1608Metric_Pad0.98x0.95mm_HandSolder, F.Cu at (141.2, 143.7)
- added R404: 100K, Resistor_SMD:R_0603_1608Metric_Pad0.98x0.95mm_HandSolder, F.Cu at (157.9, 153.0)
- added R405: 100K, Resistor_SMD:R_0603_1608Metric_Pad0.98x0.95mm_HandSolder, F.Cu at (119.2, 143.9)
- added R406: 100K, Resistor_SMD:R_0603_1608Metric_Pad0.98x0.95mm_HandSolder, F.Cu at (134.8, 143.7)
- added R407: 100K, Resistor_SMD:R_0603_1608Metric_Pad0.98x0.95mm_HandSolder, F.Cu at (183.6, 143.7)
- added R408: 100K, Resistor_SMD:R_0603_1608Metric_Pad0.98x0.95mm_HandSolder, F.Cu at (161.1, 153.0)
- added R409: 100K, Resistor_SMD:R_0603_1608Metric_Pad0.98x0.95mm_HandSolder, F.Cu at (116.0, 143.9)
- added R410: 100K, Resistor_SMD:R_0603_1608Metric_Pad0.98x0.95mm_HandSolder, F.Cu at (161.1, 144.3)
- added R411: 1K, Resistor_SMD:R_0603_1608Metric_Pad0.98x0.95mm_HandSolder, F.Cu at (151.4, 152.8)
- added R412: 1K, Resistor_SMD:R_0603_1608Metric_Pad0.98x0.95mm_HandSolder, F.Cu at (190.1, 143.7)
- added R413: 470, Resistor_SMD:R_0603_1608Metric_Pad0.98x0.95mm_HandSolder, F.Cu at (149.0, 159.7)
- added R414: 100K, Resistor_SMD:R_0603_1608Metric_Pad0.98x0.95mm_HandSolder, F.Cu at (149.0, 164.5)
- added R415: 470, Resistor_SMD:R_0603_1608Metric_Pad0.98x0.95mm_HandSolder, F.Cu at (167.4, 163.5)
- added R416: 100K, Resistor_SMD:R_0603_1608Metric_Pad0.98x0.95mm_HandSolder, F.Cu at (161.1, 163.5)
- added R417: 20K, Resistor_SMD:R_0603_1608Metric_Pad0.98x0.95mm_HandSolder, F.Cu at (145.9, 164.5)
- added R418: 20K, Resistor_SMD:R_0603_1608Metric_Pad0.98x0.95mm_HandSolder, F.Cu at (164.3, 163.5)
- added R501: 100K, Resistor_SMD:R_0603_1608Metric_Pad0.98x0.95mm_HandSolder, F.Cu at (149.0, 187.8)
- added R502: 100K, Resistor_SMD:R_0603_1608Metric_Pad0.98x0.95mm_HandSolder, F.Cu at (161.1, 192.9)
- added R503: 100K, Resistor_SMD:R_0603_1608Metric_Pad0.98x0.95mm_HandSolder, F.Cu at (141.2, 187.8)
- added R504: 100K, Resistor_SMD:R_0603_1608Metric_Pad0.98x0.95mm_HandSolder, F.Cu at (157.9, 197.1)
- added R505: 100K, Resistor_SMD:R_0603_1608Metric_Pad0.98x0.95mm_HandSolder, F.Cu at (119.2, 188.1)
- added R506: 100K, Resistor_SMD:R_0603_1608Metric_Pad0.98x0.95mm_HandSolder, F.Cu at (134.8, 187.8)
- added R507: 100K, Resistor_SMD:R_0603_1608Metric_Pad0.98x0.95mm_HandSolder, F.Cu at (183.6, 187.8)
- added R508: 100K, Resistor_SMD:R_0603_1608Metric_Pad0.98x0.95mm_HandSolder, F.Cu at (161.1, 197.1)
- added R509: 100K, Resistor_SMD:R_0603_1608Metric_Pad0.98x0.95mm_HandSolder, F.Cu at (116.0, 188.1)
- added R510: 100K, Resistor_SMD:R_0603_1608Metric_Pad0.98x0.95mm_HandSolder, F.Cu at (161.1, 188.4)
- added R511: 1K, Resistor_SMD:R_0603_1608Metric_Pad0.98x0.95mm_HandSolder, F.Cu at (151.4, 197.0)
- added R512: 1K, Resistor_SMD:R_0603_1608Metric_Pad0.98x0.95mm_HandSolder, F.Cu at (190.1, 187.8)
- added R513: 470, Resistor_SMD:R_0603_1608Metric_Pad0.98x0.95mm_HandSolder, F.Cu at (149.0, 203.8)
- added R514: 100K, Resistor_SMD:R_0603_1608Metric_Pad0.98x0.95mm_HandSolder, F.Cu at (149.0, 208.6)
- added R515: 470, Resistor_SMD:R_0603_1608Metric_Pad0.98x0.95mm_HandSolder, F.Cu at (167.4, 207.6)
- added R516: 100K, Resistor_SMD:R_0603_1608Metric_Pad0.98x0.95mm_HandSolder, F.Cu at (161.1, 207.6)
- added R517: 20K, Resistor_SMD:R_0603_1608Metric_Pad0.98x0.95mm_HandSolder, F.Cu at (145.9, 208.6)
- added R518: 20K, Resistor_SMD:R_0603_1608Metric_Pad0.98x0.95mm_HandSolder, F.Cu at (164.3, 207.6)
- added RV401: B100K, R0904NB10KL-25KQ:V2_TRIM_R0904NB10KL-25KQ-, B.Cu at (125.6, 168.5)
- added RV402: B100K, R0904NB10KL-25KQ:V2_TRIM_R0904NB10KL-25KQ-, B.Cu at (167.1, 168.5)
- added RV403: B100K, R0904NB10KL-25KQ:V2_TRIM_R0904NB10KL-25KQ-, B.Cu at (142.9, 174.5)
- added RV404: B100K, R0904NB10KL-25KQ:V2_TRIM_R0904NB10KL-25KQ-, B.Cu at (184.4, 174.5)
- added RV501: B100K, R0904NB10KL-25KQ:V2_TRIM_R0904NB10KL-25KQ-, B.Cu at (125.6, 212.6)
- added RV502: B100K, R0904NB10KL-25KQ:V2_TRIM_R0904NB10KL-25KQ-, B.Cu at (167.1, 212.6)
- added RV503: B100K, R0904NB10KL-25KQ:V2_TRIM_R0904NB10KL-25KQ-, B.Cu at (142.9, 218.6)
- added RV504: B100K, R0904NB10KL-25KQ:V2_TRIM_R0904NB10KL-25KQ-, B.Cu at (184.4, 218.6)
- added U401: MCP6004, Package_SO:TSSOP-14_4.4x5mm_P0.65mm, F.Cu at (155.1, 146.2)
- added U402: TL072, Package_SO:SOIC-8_3.9x4.9mm_P1.27mm, F.Cu at (155.0, 162.0)
- added U501: MCP6004, Package_SO:TSSOP-14_4.4x5mm_P0.65mm, F.Cu at (155.1, 190.4)
- added U502: TL072, Package_SO:SOIC-8_3.9x4.9mm_P1.27mm, F.Cu at (155.0, 206.1)
Connections:
- net /2xAttenuverters1/2xAttenuverters2_1_Out renamed /2xAttenuverters1/2xAttenuverters1_1_Out
- net /2xAttenuverters1/2xAttenuverters2_2_Out renamed /2xAttenuverters1/2xAttenuverters1_2_Out
- D301 pad 2: /2xAttenuverters1/2xAttenuverters2_1_In -> /2xAttenuverters1/2xAttenuverters1_1_In
- D303 pad 2: /2xAttenuverters1/2xAttenuverters2_2_In -> /2xAttenuverters1/2xAttenuverters1_2_In
- H301 pad 1: /2xAttenuverters1/2xAttenuverters2_1_In -> /2xAttenuverters1/2xAttenuverters1_1_In
- H303 pad 1: /2xAttenuverters1/2xAttenuverters2_2_In -> /2xAttenuverters1/2xAttenuverters1_2_In
- R301 pad 1: /2xAttenuverters1/2xAttenuverters2_1_In -> /2xAttenuverters1/2xAttenuverters1_1_In
- R302 pad 1: /2xAttenuverters1/2xAttenuverters2_2_In -> /2xAttenuverters1/2xAttenuverters1_2_In
- RV301 pad 1: /+4.5V -> /2xAttenuverters1/2xAttenuverters1_1_In
- RV301 pad 3: /2xAttenuverters1/2xAttenuverters2_1_In -> /+4.5V
- RV302 pad 1: /+4.5V -> /2xAttenuverters1/2xAttenuverters1_2_In
- RV302 pad 3: /2xAttenuverters1/2xAttenuverters2_2_In -> /+4.5V
- RV303 pad 1: /GND -> /+9V
- RV303 pad 3: /+9V -> /GND
- RV304 pad 1: /GND -> /+9V
- RV304 pad 3: /+9V -> /GND
Routing:
- net /+9V: track 131.2 -> 681.3 mm, vias 6 -> 18
- net /+4.5V: track 188.4 -> 535.5 mm, vias 14 -> 36
- net Net-(C503-Pad2): track 0.00 -> 132.0 mm, vias 0 -> 2
- net Net-(C403-Pad2): track 0.00 -> 132.0 mm, vias 0 -> 2
- net Net-(C504-Pad2): track 0.00 -> 129.4 mm, vias 0 -> 2
- net Net-(C404-Pad2): track 0.00 -> 129.4 mm, vias 0 -> 2
- net /2xAttenuverters2/2xAttenuverters1_1_In: track 0.00 -> 70.7 mm
- net /2xAttenuverters1/2xAttenuverters1_1_In: track 0.00 -> 70.7 mm
- net /2xAttenuverters3/2xAttenuverters1_1_In: track 0.00 -> 70.7 mm
- net Net-(R505-Pad2): track 0.00 -> 64.2 mm
- net Net-(R405-Pad2): track 0.00 -> 64.2 mm
- net Net-(RV401-Pad2): track 0.00 -> 60.4 mm
- net Net-(RV501-Pad2): track 0.00 -> 60.2 mm
- net /2xAttenuverters1/2xAttenuverters2_1_In: track 54.4 -> 0.00 mm
- net /2xAttenuverters1/2xAttenuverters2_2_In: track 53.6 -> 0.00 mm, vias 2 -> 0
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
Commit message: VCF schem capture
Parts:
- removed the ? at (378.4, 21.7) (x2)
- added ? (x3): , Graphics, B.Cu at (378.4, 21.7)
- added C201: 470p, Capacitor_SMD:C_0603_1608Metric_Pad1.08x0.95mm_HandSolder, F.Cu at (611.5, 44.7)
- added C601: 100n, Capacitor_SMD:C_0603_1608Metric_Pad1.08x0.95mm_HandSolder, F.Cu at (621.9, 11.1)
- added C602: 220p, Capacitor_SMD:C_0603_1608Metric_Pad1.08x0.95mm_HandSolder, F.Cu at (625.0, -2.29)
- added C603: 1.2n, Capacitor_SMD:C_0603_1608Metric_Pad1.08x0.95mm_HandSolder, F.Cu at (629.4, 0.21)
- added C604: 1.2n, Capacitor_SMD:C_0603_1608Metric_Pad1.08x0.95mm_HandSolder, F.Cu at (600.4, 23.5)
- added C605: 220p, Capacitor_SMD:C_0603_1608Metric_Pad1.08x0.95mm_HandSolder, F.Cu at (621.9, 13.6)
- added C606: 100n, Capacitor_SMD:C_0603_1608Metric_Pad1.08x0.95mm_HandSolder, F.Cu at (628.7, 5.24)
- added C607: 1.2n, Capacitor_SMD:C_0603_1608Metric_Pad1.08x0.95mm_HandSolder, F.Cu at (625.5, 16.2)
- added C608: 220p, Capacitor_SMD:C_0603_1608Metric_Pad1.08x0.95mm_HandSolder, F.Cu at (604.7, 21.0)
- added C609: 100n, Capacitor_SMD:C_0603_1608Metric_Pad1.08x0.95mm_HandSolder, F.Cu at (638.1, 2.73)
- added C610: 1.2n, Capacitor_SMD:C_0603_1608Metric_Pad1.08x0.95mm_HandSolder, F.Cu at (626.3, 10.3)
- added C611: 100n, Capacitor_SMD:C_0603_1608Metric_Pad1.08x0.95mm_HandSolder, F.Cu at (625.0, 2.73)
- added C612: 100n, Capacitor_SMD:C_0603_1608Metric_Pad1.08x0.95mm_HandSolder, F.Cu at (626.3, 12.8)
- added C613: 100n, Capacitor_SMD:C_0603_1608Metric_Pad1.08x0.95mm_HandSolder, F.Cu at (626.3, 7.75)
- added C614: 220p, Capacitor_SMD:C_0603_1608Metric_Pad1.08x0.95mm_HandSolder, F.Cu at (630.6, 10.3)
- added C615: 100n, Capacitor_SMD:C_0603_1608Metric_Pad1.08x0.95mm_HandSolder, F.Cu at (638.1, 0.21)
- added C616: 100n, Capacitor_SMD:C_0603_1608Metric_Pad1.08x0.95mm_HandSolder, F.Cu at (604.7, 23.5)
- added C701: 100n, Capacitor_SMD:C_0603_1608Metric_Pad1.08x0.95mm_HandSolder, F.Cu at (665.1, 12.9)
- added C702: 100n, Capacitor_SMD:C_0603_1608Metric_Pad1.08x0.95mm_HandSolder, F.Cu at (677.9, 3.17)
- added C801: 100n, Capacitor_SMD:C_0603_1608Metric_Pad1.08x0.95mm_HandSolder, F.Cu at (648.3, -37.0)
- added C802: 100n, Capacitor_SMD:C_0603_1608Metric_Pad1.08x0.95mm_HandSolder, F.Cu at (634.7, -21.8)
- added C803: 100n, Capacitor_SMD:C_0603_1608Metric_Pad1.08x0.95mm_HandSolder, F.Cu at (633.8, -31.9)
- added C804: 100n, Capacitor_SMD:C_0603_1608Metric_Pad1.08x0.95mm_HandSolder, F.Cu at (628.0, -16.9)
- added C805: 100n, Capacitor_SMD:C_0603_1608Metric_Pad1.08x0.95mm_HandSolder, F.Cu at (643.4, -29.4)
- added C806: 100n, Capacitor_SMD:C_0603_1608Metric_Pad1.08x0.95mm_HandSolder, F.Cu at (648.3, -42.0)
- added D601: D, Diode_SMD:D_SOD-323_HandSoldering, F.Cu at (620.3, 0.88)
- added D602: D, Diode_SMD:D_SOD-323_HandSoldering, F.Cu at (620.3, -2.08)
- added D603: D_TVS, Diode_SMD:D_SOD-323_HandSoldering, F.Cu at (603.4, 18.3)
- added D604: D_Zener, Diode_SMD:D_SOD-123, F.Cu at (595.3, 19.8)
- added D605: D_Zener, Diode_SMD:D_SOD-123, F.Cu at (595.3, 23.1)
- added D701: D_TVS, Diode_SMD:D_SOD-323_HandSoldering, F.Cu at (668.8, 4.38)
- added D702: D_TVS, Diode_SMD:D_SOD-323_HandSoldering, F.Cu at (677.3, -2.08)
- added D703: D, Diode_SMD:D_SOD-323_HandSoldering, F.Cu at (660.4, 8.07)
- added D704: D, Diode_SMD:D_SOD-323_HandSoldering, F.Cu at (660.4, 11.0)
- added D801: D_TVS, Diode_SMD:D_SOD-323_HandSoldering, F.Cu at (595.0, -8.95)
- added D802: D_TVS, Diode_SMD:D_SOD-323_HandSoldering, F.Cu at (595.0, -11.9)
- added D803: D_TVS, Diode_SMD:D_SOD-323_HandSoldering, F.Cu at (600.0, -8.95)
- added D804: D_TVS, Diode_SMD:D_SOD-323_HandSoldering, F.Cu at (600.0, -11.9)
- added H601: Main_Out, MountingHole:MountingHole_4.3mm_M4_Pad_TopBottom, F.Cu at (606.0, 11.7)
- added H701: Freq_In, MountingHole:MountingHole_4.3mm_M4_Pad_TopBottom, F.Cu at (652.8, 11.7)
- added H702: Res_In, MountingHole:MountingHole_4.3mm_M4_Pad_TopBottom, F.Cu at (661.2, 1.52)
- added H801: HP_Out, MountingHole:MountingHole_4.3mm_M4_Pad_TopBottom, F.Cu at (620.7, -13.0)
- added H802: UBP_Out, MountingHole:MountingHole_4.3mm_M4_Pad_TopBottom, F.Cu at (610.6, -13.0)
- added H803: LBP_Out, MountingHole:MountingHole_4.3mm_M4_Pad_TopBottom, F.Cu at (627.5, -23.2)
- added H804: LP_Out, MountingHole:MountingHole_4.3mm_M4_Pad_TopBottom, F.Cu at (636.7, -38.2)
- added Q201: Q_PNP_BEC, Package_TO_SOT_SMD:SOT-23_Handsoldering, F.Cu at (612.6, 38.6)
- added R201: 30K, Resistor_SMD:R_0603_1608Metric_Pad0.98x0.95mm_HandSolder, F.Cu at (623.6, 32.6)
- added R202: 8.2K, Resistor_SMD:R_0603_1608Metric_Pad0.98x0.95mm_HandSolder, F.Cu at (628.0, 30.1)
- added R203: 100K, Resistor_SMD:R_0603_1608Metric_Pad0.98x0.95mm_HandSolder, F.Cu at (594.6, 49.1)
- added R204: 100K, Resistor_SMD:R_0603_1608Metric_Pad0.98x0.95mm_HandSolder, F.Cu at (611.5, 42.2)
- added R205: 10K, Resistor_SMD:R_0603_1608Metric_Pad0.98x0.95mm_HandSolder, F.Cu at (622.3, 37.6)
- added R206: 30K, Resistor_SMD:R_0603_1608Metric_Pad0.98x0.95mm_HandSolder, F.Cu at (615.9, 42.2)
- added R207: 1K, Resistor_SMD:R_0603_1608Metric_Pad0.98x0.95mm_HandSolder, F.Cu at (615.9, 44.7)
- added R208: 5K, Resistor_SMD:R_0603_1608Metric_Pad0.98x0.95mm_HandSolder, F.Cu at (623.6, 35.1)
- added R209: 680, Resistor_SMD:R_0603_1608Metric_Pad0.98x0.95mm_HandSolder, F.Cu at (611.5, 47.2)
- added R210: 30K, Resistor_SMD:R_0603_1608Metric_Pad0.98x0.95mm_HandSolder, F.Cu at (623.6, 30.1)
- added R211: 8.2K, Resistor_SMD:R_0603_1608Metric_Pad0.98x0.95mm_HandSolder, F.Cu at (620.2, 40.1)
- added R212: 20K, Resistor_SMD:R_0603_1608Metric_Pad0.98x0.95mm_HandSolder, F.Cu at (618.0, 37.6)
- added R601: 1M, Resistor_SMD:R_0603_1608Metric_Pad0.98x0.95mm_HandSolder, F.Cu at (633.7, 0.21)
- added R602: 33K, Resistor_SMD:R_0603_1608Metric_Pad0.98x0.95mm_HandSolder, F.Cu at (613.4, 23.1)
- added R603: 33K, Resistor_SMD:R_0603_1608Metric_Pad0.98x0.95mm_HandSolder, F.Cu at (617.6, 8.62)
- added R604: 33K, Resistor_SMD:R_0603_1608Metric_Pad0.98x0.95mm_HandSolder, F.Cu at (633.0, 5.24)
- added R605: 33K, Resistor_SMD:R_0603_1608Metric_Pad0.98x0.95mm_HandSolder, F.Cu at (642.4, -2.29)
- added R606: 200K, Resistor_SMD:R_0603_1608Metric_Pad0.98x0.95mm_HandSolder, F.Cu at (609.1, 23.1)
- added R607: 33K, Resistor_SMD:R_0603_1608Metric_Pad0.98x0.95mm_HandSolder, F.Cu at (616.8, 18.0)
- added R608: 33K, Resistor_SMD:R_0603_1608Metric_Pad0.98x0.95mm_HandSolder, F.Cu at (600.4, 21.0)
- added R609: 33K, Resistor_SMD:R_0603_1608Metric_Pad0.98x0.95mm_HandSolder, F.Cu at (613.4, 20.6)
- added R610: 33K, Resistor_SMD:R_0603_1608Metric_Pad0.98x0.95mm_HandSolder, F.Cu at (638.1, -2.29)
- added R611: 33K, Resistor_SMD:R_0603_1608Metric_Pad0.98x0.95mm_HandSolder, F.Cu at (620.0, 3.60)
- added R612: 22K, Resistor_SMD:R_0603_1608Metric_Pad0.98x0.95mm_HandSolder, F.Cu at (613.2, 12.9)
- added R613: 33K, Resistor_SMD:R_0603_1608Metric_Pad0.98x0.95mm_HandSolder, F.Cu at (613.2, 10.4)
- added R614: 220, Resistor_SMD:R_0603_1608Metric_Pad0.98x0.95mm_HandSolder, F.Cu at (629.4, 2.73)
- added R615: 10K, Resistor_SMD:R_0603_1608Metric_Pad0.98x0.95mm_HandSolder, F.Cu at (629.4, -2.29)
- added R616: 10K, Resistor_SMD:R_0603_1608Metric_Pad0.98x0.95mm_HandSolder, F.Cu at (617.8, 20.5)
- added R617: 10K, Resistor_SMD:R_0603_1608Metric_Pad0.98x0.95mm_HandSolder, F.Cu at (617.6, 13.6)
- added R618: 10K, Resistor_SMD:R_0603_1608Metric_Pad0.98x0.95mm_HandSolder, F.Cu at (613.2, 15.4)
- added R619: 220, Resistor_SMD:R_0603_1608Metric_Pad0.98x0.95mm_HandSolder, F.Cu at (617.8, 23.0)
- added R620: 10K, Resistor_SMD:R_0603_1608Metric_Pad0.98x0.95mm_HandSolder, F.Cu at (633.7, 2.73)
- added R621: 3.3K, Resistor_SMD:R_0603_1608Metric_Pad0.98x0.95mm_HandSolder, F.Cu at (633.7, -2.29)
- added R622: 1K, Resistor_SMD:R_0603_1608Metric_Pad0.98x0.95mm_HandSolder, F.Cu at (609.1, 20.6)
- added R623: 33K, Resistor_SMD:R_0603_1608Metric_Pad0.98x0.95mm_HandSolder, F.Cu at (624.3, 5.24)
- added R624: 330K, Resistor_SMD:R_0603_1608Metric_Pad0.98x0.95mm_HandSolder, F.Cu at (608.1, 18.1)
- added R625: 33K, Resistor_SMD:R_0603_1608Metric_Pad0.98x0.95mm_HandSolder, F.Cu at (625.0, 0.21)
- added R626: 33K, Resistor_SMD:R_0603_1608Metric_Pad0.98x0.95mm_HandSolder, F.Cu at (617.6, 11.1)
- added R627: 30K, Resistor_SMD:R_0603_1608Metric_Pad0.98x0.95mm_HandSolder, F.Cu at (620.0, 6.12)
- added R628: 200K, Resistor_SMD:R_0603_1608Metric_Pad0.98x0.95mm_HandSolder, F.Cu at (621.2, 16.2)
- added R629: 220, Resistor_SMD:R_0603_1608Metric_Pad0.98x0.95mm_HandSolder, F.Cu at (630.6, 7.75)
- added R630: 33K, Resistor_SMD:R_0603_1608Metric_Pad0.98x0.95mm_HandSolder, F.Cu at (613.2, 7.92)
- added R631: 220, Resistor_SMD:R_0603_1608Metric_Pad0.98x0.95mm_HandSolder, F.Cu at (621.9, 8.62)
- added R632: 3.3K, Resistor_SMD:R_0603_1608Metric_Pad0.98x0.95mm_HandSolder, F.Cu at (612.5, 18.1)
- added R701: 100K, Resistor_SMD:R_0603_1608Metric_Pad0.98x0.95mm_HandSolder, F.Cu at (665.1, 7.86)
- added R702: 100K, Resistor_SMD:R_0603_1608Metric_Pad0.98x0.95mm_HandSolder, F.Cu at (676.9, 0.66)
- added R703: 1K, Resistor_SMD:R_0603_1608Metric_Pad0.98x0.95mm_HandSolder, F.Cu at (660.0, 13.8)
- added R704: 1K, Resistor_SMD:R_0603_1608Metric_Pad0.98x0.95mm_HandSolder, F.Cu at (664.4, 15.4)
- added R705: 10K, Resistor_SMD:R_0603_1608Metric_Pad0.98x0.95mm_HandSolder, F.Cu at (669.4, 7.11)
- added R706: 5.6K, Resistor_SMD:R_0603_1608Metric_Pad0.98x0.95mm_HandSolder, F.Cu at (669.4, 9.62)
- added R707: 1K, Resistor_SMD:R_0603_1608Metric_Pad0.98x0.95mm_HandSolder, F.Cu at (673.5, 4.16)
- added R708: 1K, Resistor_SMD:R_0603_1608Metric_Pad0.98x0.95mm_HandSolder, F.Cu at (665.1, 10.4)
- added R801: 1K, Resistor_SMD:R_0603_1608Metric_Pad0.98x0.95mm_HandSolder, F.Cu at (634.7, -26.8)
- added R802: 1K, Resistor_SMD:R_0603_1608Metric_Pad0.98x0.95mm_HandSolder, F.Cu at (634.7, -29.4)
- added R803: 1K, Resistor_SMD:R_0603_1608Metric_Pad0.98x0.95mm_HandSolder, F.Cu at (643.9, -34.5)
- added R804: 1K, Resistor_SMD:R_0603_1608Metric_Pad0.98x0.95mm_HandSolder, F.Cu at (648.3, -39.5)
- added R805: 200K, Resistor_SMD:R_0603_1608Metric_Pad0.98x0.95mm_HandSolder, F.Cu at (639.1, -26.8)
- added R806: 200K, Resistor_SMD:R_0603_1608Metric_Pad0.98x0.95mm_HandSolder, F.Cu at (652.6, -39.5)
- added R807: 200K, Resistor_SMD:R_0603_1608Metric_Pad0.98x0.95mm_HandSolder, F.Cu at (642.5, -31.9)
- added R808: 200K, Resistor_SMD:R_0603_1608Metric_Pad0.98x0.95mm_HandSolder, F.Cu at (628.0, -14.4)
- added R809: 100K, Resistor_SMD:R_0603_1608Metric_Pad0.98x0.95mm_HandSolder, F.Cu at (643.9, -39.5)
- added R810: 100K, Resistor_SMD:R_0603_1608Metric_Pad0.98x0.95mm_HandSolder, F.Cu at (639.1, -29.4)
- added R811: 100K, Resistor_SMD:R_0603_1608Metric_Pad0.98x0.95mm_HandSolder, F.Cu at (648.3, -34.5)
- added R812: 100K, Resistor_SMD:R_0603_1608Metric_Pad0.98x0.95mm_HandSolder, F.Cu at (643.9, -37.0)
- added R813: 100K, Resistor_SMD:R_0603_1608Metric_Pad0.98x0.95mm_HandSolder, F.Cu at (634.7, -24.3)
- added R814: 100K, Resistor_SMD:R_0603_1608Metric_Pad0.98x0.95mm_HandSolder, F.Cu at (652.6, -42.0)
- added R815: 100K, Resistor_SMD:R_0603_1608Metric_Pad0.98x0.95mm_HandSolder, F.Cu at (638.1, -31.9)
- added R816: 100K, Resistor_SMD:R_0603_1608Metric_Pad0.98x0.95mm_HandSolder, F.Cu at (643.9, -42.0)
- added RV201: 100K multiturn, Potentiometer_SMD:Potentiometer_Bourns_3314J_Vertical, F.Cu at (618.4, 32.6)
- added RV202: 1K, Potentiometer_SMD:Potentiometer_Bourns_3314J_Vertical, F.Cu at (612.4, 32.6)
- added RV203: 1K, Potentiometer_SMD:Potentiometer_Bourns_3314J_Vertical, F.Cu at (595.5, 44.0)
- added RV801: B100K, R0904NB10KL-25KQ:V2_TRIM_R0904NB10KL-25KQ-, F.Cu at (625.1, -37.0)
- added RV802: B100K, R0904NB10KL-25KQ:V2_TRIM_R0904NB10KL-25KQ-, F.Cu at (599.0, -37.0)
- added RV803: B100K, R0904NB10KL-25KQ:V2_TRIM_R0904NB10KL-25KQ-, F.Cu at (599.0, -22.0)
- added RV804: B100K, R0904NB10KL-25KQ:V2_TRIM_R0904NB10KL-25KQ-, F.Cu at (612.0, -37.0)
- added U201: LM13700, Package_SO:SOIC-16_3.9x9.9mm_P1.27mm, F.Cu at (596.7, 34.5)
- added U202: MCP6004, Package_SO:SOIC-14_3.9x8.7mm_P1.27mm, F.Cu at (605.1, 44.1)
- added U203: MCP6004, Package_SO:SOIC-14_3.9x8.7mm_P1.27mm, F.Cu at (605.1, 33.9)
- added U601: TL074, Package_SO:SOIC-14_3.9x8.7mm_P1.27mm, F.Cu at (596.7, 13.0)
- added U602: TL074, Package_SO:SOIC-14_3.9x8.7mm_P1.27mm, F.Cu at (605.1, 1.55)
- added U603: SSI2164, Package_SO:SOIC-16_3.9x9.9mm_P1.27mm, F.Cu at (596.7, 2.17)
- added U604: TL074, Package_SO:SOIC-14_3.9x8.7mm_P1.27mm, F.Cu at (613.6, 1.55)
- added U701: TL074, Package_SO:SOIC-14_3.9x8.7mm_P1.27mm, F.Cu at (651.9, 1.55)
- added U702: TL072, Package_SO:SOIC-8_3.9x4.9mm_P1.27mm, F.Cu at (670.5, -0.33)
- added U801: TL074, Package_SO:SOIC-14_3.9x8.7mm_P1.27mm, F.Cu at (609.7, -23.2)
- added U802: TL074, Package_SO:SOIC-14_3.9x8.7mm_P1.27mm, F.Cu at (618.2, -23.2)
- C301, C302, C303, C304, C401, C402, C403, C404, C501, C502, C503, C504: value 30p -> 10p
- U301, U401, U501: footprint Package_SO:TSSOP-14_4.4x5mm_P0.65mm -> Package_SO:SOIC-14_3.9x8.7mm_P1.27mm
Connections:
- net /2xAttenuverters1/2xAttenuverters1_1_In renamed /2xAttenuverters1/_1_In
- net /2xAttenuverters1/2xAttenuverters1_1_Out renamed /2xAttenuverters1/_1_Out
- net /2xAttenuverters1/2xAttenuverters1_2_In renamed /2xAttenuverters1/_2_In
- net /2xAttenuverters1/2xAttenuverters1_2_Out renamed /2xAttenuverters1/_2_Out
- net /2xAttenuverters2/2xAttenuverters1_1_In renamed /2xAttenuverters2/_1_In
- net /2xAttenuverters2/2xAttenuverters1_1_Out renamed /2xAttenuverters2/_1_Out
- net /2xAttenuverters2/2xAttenuverters1_2_In renamed /2xAttenuverters2/_2_In
- net /2xAttenuverters2/2xAttenuverters1_2_Out renamed /2xAttenuverters2/_2_Out
- net /2xAttenuverters3/2xAttenuverters1_1_In renamed /2xAttenuverters3/_1_In
- net /2xAttenuverters3/2xAttenuverters1_1_Out renamed /2xAttenuverters3/_1_Out
- net /2xAttenuverters3/2xAttenuverters1_2_In renamed /2xAttenuverters3/_2_In
- net /2xAttenuverters3/2xAttenuverters1_2_Out renamed /2xAttenuverters3/_2_Out
Routing:
- net /+9V: track 681.3 -> 678.5 mm
- net Net-(C303-Pad1): track 44.5 -> 42.3 mm
- net Net-(C403-Pad1): track 44.5 -> 42.3 mm
- net Net-(C503-Pad1): track 44.5 -> 42.3 mm
- net Net-(C502-Pad2): track 10.2 -> 8.54 mm
- net Net-(C302-Pad2): track 10.2 -> 8.54 mm
- net Net-(C402-Pad2): track 10.2 -> 8.54 mm
- net Net-(C501-Pad1): track 18.5 -> 20.2 mm
- net Net-(C401-Pad1): track 18.5 -> 20.2 mm
- net Net-(C301-Pad1): track 18.5 -> 20.2 mm
- net Net-(RV401-Pad2): track 60.4 -> 58.9 mm
- net Net-(RV301-Pad2): track 60.4 -> 58.9 mm
- net Net-(C403-Pad2): track 132.0 -> 130.6 mm
- net Net-(C303-Pad2): track 132.0 -> 130.6 mm
- net Net-(C503-Pad2): track 132.0 -> 130.6 mm
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
Commit message: Start VCF layout
Parts:
- added D606: D_TVS, Diode_SMD:D_SOD-323_HandSoldering, F.Cu at (28.4, 90.4)
- added H602: In, MountingHole:MountingHole_4.3mm_M4_Pad_TopBottom, B.Cu at (35.7, 91.7)
- H601, H701, H702, H801, H802, H803, H804, RV801, RV802, RV803, RV804: moved to B.Cu
- moved R804 629.0 mm to (38.3, 114.1), turned to 90 degrees
- moved D701 628.9 mm to (45.8, 90.4), turned to -90 degrees
- moved C805 622.7 mm to (38.4, 118.0), turned to 90 degrees
- moved C702 621.8 mm to (63.7, 100.5), turned to 90 degrees
- moved H804 618.5 mm to (35.7, 107.7), turned to 180 degrees
- moved R808 615.0 mm to (25.1, 106.8), turned to 90 degrees
- moved R807 614.7 mm to (43.6, 106.8), turned to 90 degrees
- moved R803 612.3 mm to (50.0, 114.1), turned to 90 degrees
- moved C804 606.8 mm to (35.5, 114.1), turned to -90 degrees
- moved H701 605.2 mm to (52.9, 91.7), turned to 180 degrees
- moved D702 600.2 mm to (84.2, 90.4), turned to -90 degrees
- moved RV804 598.9 mm to (35.6, 125.6), turned to 180 degrees
- moved C803 598.8 mm to (53.0, 114.1), turned to -90 degrees
- moved U702 594.7 mm to (84.2, 99.5)
- moved H702 591.0 mm to (77.1, 91.6), turned to 180 degrees
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Connections:
- net /2xAttenuverters1/_1_In renamed /2xAttenuverters1/VCF Audio Outs_1_In
- net /2xAttenuverters1/_1_Out renamed /2xAttenuverters1/VCF Audio Outs_1_Out
- net /2xAttenuverters1/_2_In renamed /2xAttenuverters1/VCF Audio Outs_2_In
- net /2xAttenuverters1/_2_Out renamed /2xAttenuverters1/VCF Audio Outs_2_Out
- net /2xAttenuverters2/_1_In renamed /2xAttenuverters2/VCF Audio Outs_1_In
- net /2xAttenuverters2/_1_Out renamed /2xAttenuverters2/VCF Audio Outs_1_Out
- net /2xAttenuverters2/_2_In renamed /2xAttenuverters2/VCF Audio Outs_2_In
- net /2xAttenuverters2/_2_Out renamed /2xAttenuverters2/VCF Audio Outs_2_Out
- net /2xAttenuverters3/_1_In renamed /2xAttenuverters3/VCF Audio Outs_1_In
- net /2xAttenuverters3/_1_Out renamed /2xAttenuverters3/VCF Audio Outs_1_Out
- net /2xAttenuverters3/_2_In renamed /2xAttenuverters3/VCF Audio Outs_2_In
- net /2xAttenuverters3/_2_Out renamed /2xAttenuverters3/VCF Audio Outs_2_Out
- C603 pad 2: /VCF/+4.5V -> /+4.5V
- C604 pad 2: /VCF/+4.5V -> /+4.5V
- C607 pad 2: /VCF/+4.5V -> /+4.5V
- C610 pad 2: /VCF/+4.5V -> /+4.5V
- C612 pad 1: /VCF/GND -> /GND
- C612 pad 2: /VCF/+9V -> /+9V
- C613 pad 1: /VCF/GND -> /GND
- C613 pad 2: /VCF/+9V -> /+9V
- C615 pad 1: /VCF/+9V -> /+9V
- C615 pad 2: /VCF/GND -> /GND
- C616 pad 1: /VCF/GND -> /GND
- C616 pad 2: /VCF/+4.5V -> /+4.5V
- C701 pad 1: /VCF/GND -> /GND
- C701 pad 2: /VCF/+9V -> /+9V
- C702 pad 1: /VCF/GND -> /GND
- C702 pad 2: /VCF/+9V -> /+9V
- C805 pad 1: /VCF/GND -> /GND
- C805 pad 2: /VCF/+9V -> /+9V
- C806 pad 1: /VCF/GND -> /GND
- C806 pad 2: /VCF/+9V -> /+9V
- D603 pad 1: /VCF/GND -> /GND
- D605 pad 1: /VCF/+4.5V -> /+4.5V
- D701 pad 1: /VCF/GND -> /GND
- D702 pad 1: /VCF/GND -> /GND
- D801 pad 1: /VCF/GND -> /GND
- D802 pad 1: /VCF/GND -> /GND
- D803 pad 1: /VCF/GND -> /GND
- D804 pad 1: /VCF/GND -> /GND
- R601 pad 2: /VCF/GND -> /GND
- R604 pad 1: /VCF/+4.5V -> /+4.5V
- R606 pad 2: /VCF/+4.5V -> /+4.5V
- R608 pad 1: /VCF/+4.5V -> /+4.5V
- R628 pad 2: /VCF/GND -> /GND
- R701 pad 2: /VCF/+4.5V -> /+4.5V
- R702 pad 2: /VCF/+4.5V -> /+4.5V
- R706 pad 1: /VCF/+4.5V -> /+4.5V
- R805 pad 2: /VCF/GND -> /GND
- R806 pad 2: /VCF/GND -> /GND
- R807 pad 2: /VCF/GND -> /GND
- R808 pad 2: /VCF/GND -> /GND
- RV801 pad 0: /VCF/GND -> /GND
- RV801 pad 3: /VCF/+4.5V -> /+4.5V
- RV802 pad 0: /VCF/GND -> /GND
- RV802 pad 3: /VCF/+4.5V -> /+4.5V
- RV803 pad 0: /VCF/GND -> /GND
- RV803 pad 3: /VCF/+4.5V -> /+4.5V
- RV804 pad 0: /VCF/GND -> /GND
- RV804 pad 3: /VCF/+4.5V -> /+4.5V
- U601 pad 11: /VCF/GND -> /GND
- U601 pad 12: /VCF/+4.5V -> /+4.5V
- U601 pad 4: /VCF/+9V -> /+9V
- U601 pad 5: /VCF/+4.5V -> /+4.5V
- U602 pad 10: /VCF/+4.5V -> /+4.5V
- U602 pad 11: /VCF/GND -> /GND
- U602 pad 12: /VCF/+4.5V -> /+4.5V
- U602 pad 3: /VCF/+4.5V -> /+4.5V
- U602 pad 4: /VCF/+9V -> /+9V
- U602 pad 5: /VCF/+4.5V -> /+4.5V
- U603 pad 16: /VCF/+9V -> /+9V
- U603 pad 8: /VCF/+4.5V -> /+4.5V
- U603 pad 9: /VCF/GND -> /GND
- U701 pad 11: /VCF/GND -> /GND
- U701 pad 4: /VCF/+9V -> /+9V
- U701 pad 5: /VCF/+4.5V -> /+4.5V
- U702 pad 3: /VCF/+4.5V -> /+4.5V
- U702 pad 4: /VCF/GND -> /GND
- U702 pad 8: /VCF/+9V -> /+9V
- U801 pad 1: Net-(R801-Pad1) -> Net-(R802-Pad1)
- U801 pad 10: /VCF/UBP -> Net-(RV801-Pad2)
- U801 pad 11: /VCF/GND -> /GND
- U801 pad 12: Net-(RV802-Pad2) -> /VCF/HP
- U801 pad 13: Net-(R810-Pad2) -> Net-(R801-Pad1)
- U801 pad 14: /VCF/UBP_Vert -> Net-(R801-Pad1)
- U801 pad 2: Net-(R801-Pad1) -> Net-(R802-Pad1)
- U801 pad 3: /VCF/HP -> /VCF/UBP
- U801 pad 4: /VCF/+9V -> /+9V
- U801 pad 5: Net-(RV801-Pad2) -> Net-(RV802-Pad2)
- U801 pad 6: Net-(R809-Pad2) -> Net-(R810-Pad2)
- U801 pad 7: /VCF/HP_Vert -> /VCF/UBP_Vert
- U801 pad 8: Net-(R802-Pad1) -> /VCF/HP_Vert
- U801 pad 9: Net-(R802-Pad1) -> Net-(R809-Pad2)
- U802 pad 1: Net-(R803-Pad1) -> Net-(R804-Pad1)
- U802 pad 10: /VCF/LP -> Net-(RV803-Pad2)
- U802 pad 11: /VCF/GND -> /GND
- U802 pad 12: Net-(RV804-Pad2) -> /VCF/LBP
- U802 pad 13: Net-(R812-Pad2) -> Net-(R803-Pad1)
- U802 pad 14: /VCF/LP_Vert -> Net-(R803-Pad1)
- U802 pad 2: Net-(R803-Pad1) -> Net-(R804-Pad1)
- U802 pad 3: /VCF/LBP -> /VCF/LP
- U802 pad 4: /VCF/+9V -> /+9V
- U802 pad 5: Net-(RV803-Pad2) -> Net-(RV804-Pad2)
- U802 pad 6: Net-(R811-Pad2) -> Net-(R812-Pad2)
- U802 pad 7: /VCF/LBP_Vert -> /VCF/LP_Vert
- U802 pad 8: Net-(R804-Pad1) -> /VCF/LBP_Vert
- U802 pad 9: Net-(R804-Pad1) -> Net-(R811-Pad2)
