File: konstrukt-kicad6.kicad_pcb (KiCad board)
At the start: 2 copper layers, 356.9 x 210 mm, 264 parts, among them Q201 Q_PNP_BEC, U201 LM13700, U202 MCP6004, U203 MCP6004, U301 MCP6004, U302 TL072, U401 MCP6004, U402 TL072, U501 MCP6004, U502 TL072, U601 TL074, U602 TL074, U603 SSI2164, U604 TL074, U701 TL074, U702 TL072, U801 TL074, U802 TL074

Commit message: WIP VCF Layout
Parts:
- removed C609, C611: 100n, Capacitor_SMD:C_0603_1608Metric_Pad1.08x0.95mm_HandSolder
- removed U604: TL074, Package_SO:SOIC-14_3.9x8.7mm_P1.27mm
- moved R625 601.2 mm to (39.8, 137.8), turned to 90 degrees
- moved C614 594.5 mm to (50.0, 137.8), turned to 90 degrees
- moved R621 594.2 mm to (48.7, 101.8), turned to -90 degrees
- moved D602 593.4 mm to (35.5, 98.7), turned to -90 degrees
- moved C602 591.1 mm to (42.4, 97.4), turned to 90 degrees
- moved R601 589.7 mm to (52.3, 98.6), turned to -90 degrees
- moved D601 589.4 mm to (39.1, 98.7), turned to 90 degrees
- moved R618 587.6 mm to (35.5, 122.8)
- moved C610 587.0 mm to (53.3, 137.8), turned to -90 degrees
- moved R623 586.9 mm to (45.4, 101.8), turned to -90 degrees
- moved R610 585.6 mm to (63.6, 111.3), turned to -90 degrees
- moved R617 584.0 mm to (44.1, 124.0)
- moved C603 582.9 mm to (60.4, 126.6), turned to -90 degrees
- moved R605 582.1 mm to (70.8, 107.5), turned to -90 degrees
- moved C615 582.1 mm to (70.8, 130.7), turned to 90 degrees
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Connections:
- net /2xAttenuverters1/VCF Audio Outs_1_In renamed /2xAttenuverters1/VCF_1_In
- net /2xAttenuverters1/VCF Audio Outs_1_Out renamed /2xAttenuverters1/VCF_1_Out
- net /2xAttenuverters1/VCF Audio Outs_2_In renamed /2xAttenuverters1/VCF_2_In
- net /2xAttenuverters1/VCF Audio Outs_2_Out renamed /2xAttenuverters1/VCF_2_Out
- net /2xAttenuverters2/VCF Audio Outs_1_In renamed /2xAttenuverters2/VCF_1_In
- net /2xAttenuverters2/VCF Audio Outs_1_Out renamed /2xAttenuverters2/VCF_1_Out
- net /2xAttenuverters2/VCF Audio Outs_2_In renamed /2xAttenuverters2/VCF_2_In
- net /2xAttenuverters2/VCF Audio Outs_2_Out renamed /2xAttenuverters2/VCF_2_Out
- net /2xAttenuverters3/VCF Audio Outs_1_In renamed /2xAttenuverters3/VCF_1_In
- net /2xAttenuverters3/VCF Audio Outs_1_Out renamed /2xAttenuverters3/VCF_1_Out
- net /2xAttenuverters3/VCF Audio Outs_2_In renamed /2xAttenuverters3/VCF_2_In
- net /2xAttenuverters3/VCF Audio Outs_2_Out renamed /2xAttenuverters3/VCF_2_Out
- C605 pad 1: /VCF/VCA_I_Out1 -> /VCF/VCA_I_Out4
- C608 pad 1: /VCF/VCA_I_Out2 -> /VCF/VCA_I_Out3
- C614 pad 1: /VCF/VCA_I_Out3 -> /VCF/VCA_I_Out2
- R612 pad 2: /VCF/VCA_I_In4 -> /VCF/VCA_I_In1
- R613 pad 2: /VCF/VCA_I_In1 -> /VCF/VCA_I_In4
- R614 pad 1: /VCF/VCA_I_In4 -> /VCF/VCA_I_In1
- R619 pad 1: /VCF/VCA_I_In1 -> /VCF/VCA_I_In4
- R623 pad 2: /VCF/VCA_I_Out4 -> /VCF/VCA_I_Out1
- R624 pad 1: /VCF/VCA_I_Out4 -> /VCF/VCA_I_Out1
- R625 pad 2: /VCF/VCA_I_Out4 -> /VCF/VCA_I_Out1
- R626 pad 2: /VCF/VCA_I_In2 -> /VCF/VCA_I_In3
- R627 pad 1: /VCF/VCA_I_Out4 -> /VCF/VCA_I_Out1
- R629 pad 1: /VCF/VCA_I_In2 -> /VCF/VCA_I_In3
- R630 pad 2: /VCF/VCA_I_In3 -> /VCF/VCA_I_In2
- R631 pad 1: /VCF/VCA_I_In3 -> /VCF/VCA_I_In2
- U601 pad 6: /VCF/VCA_I_Out4 -> /VCF/VCA_I_Out1
- U602 pad 1: /VCF/HP -> /VCF/LP
- U602 pad 13: /VCF/VCA_I_Out3 -> Net-(R609-Pad2)
- U602 pad 14: /VCF/LP -> /VCF/HP
- U602 pad 2: Net-(R609-Pad2) -> /VCF/VCA_I_Out2
- U602 pad 6: /VCF/VCA_I_Out1 -> /VCF/VCA_I_Out3
- U602 pad 7: /VCF/UBP -> /VCF/LBP
- U602 pad 8: /VCF/LBP -> /VCF/UBP
- U602 pad 9: /VCF/VCA_I_Out2 -> /VCF/VCA_I_Out4
Routing:
- net Net-(R615-Pad2): track 0.00 -> 138.7 mm, vias 0 -> 6
- net /VCF/LP: track 0.00 -> 110.8 mm
- net /VCF/HP: track 0.00 -> 71.7 mm, vias 0 -> 4
- net /VCF/UBP: track 0.00 -> 68.2 mm, vias 0 -> 2
- net /+4.5V: track 535.6 -> 582.3 mm, vias 36 -> 42
- net /VCF/LBP: track 0.00 -> 45.2 mm, vias 0 -> 2
- net /VCF/VCA_I_Out2: track 0.00 -> 40.1 mm
- net /VCF/VCA_I_Out3: track 0.00 -> 29.9 mm, vias 0 -> 2
- net /VCF/VCA_I_Out1: track 0.00 -> 27.7 mm
- net Net-(RV801-Pad2): track 0.00 -> 24.9 mm
- net /+9V: track 678.5 -> 702.2 mm
- net Net-(RV804-Pad2): track 0.00 -> 22.7 mm
- net Net-(RV802-Pad2): track 0.00 -> 21.8 mm
- net /VCF/VCF Audio Outs/LP_Out: track 0.00 -> 19.1 mm
- net Net-(RV803-Pad2): track 0.00 -> 18.2 mm, vias 0 -> 2
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