File: konstrukt-kicad6.kicad_pcb (KiCad board)
At the start: 2 copper layers, 356.9 x 210 mm, 261 parts, among them Q201 Q_PNP_BEC, U201 LM13700, U202 MCP6004, U203 MCP6004, U301 MCP6004, U302 TL072, U401 MCP6004, U402 TL072, U501 MCP6004, U502 TL072, U601 TL074, U602 TL074, U603 SSI2164, U701 TL074, U702 TL072, U801 TL074, U802 TL074

Commit message: VCF layout wip
Parts:
- moved R609 0.25 mm to (59.1, 113.6)
- turned R707 to 180 degrees
Routing:
- net /+4.5V: track 582.3 -> 894.4 mm, vias 42 -> 65
- net /VCF/VCA_VC1: track 9.83 -> 164.7 mm, vias 2 -> 4
- net /+9V: track 702.2 -> 803.5 mm, vias 18 -> 30
- net /VCF/VCA_VC4: track 0.00 -> 90.1 mm, vias 0 -> 4
- net /VCF/UBP-LBP: track 0.00 -> 74.7 mm, vias 0 -> 5
- net /VCF/VCA_I_Out1: track 27.7 -> 86.0 mm, vias 0 -> 6
- net Net-(R615-Pad2): track 138.7 -> 187.8 mm, vias 6 -> 8
- net Net-(R620-Pad2): track 0.00 -> 33.9 mm, vias 0 -> 2
- net Net-(D703-Pad1): track 0.00 -> 32.9 mm, vias 0 -> 4
- net /VCF/VCF CV Ins/Res_In: track 0.00 -> 32.5 mm, vias 0 -> 2
- net /GND: track 27.3 -> 57.7 mm, vias 24 -> 52
- net /VCF/In: track 0.00 -> 30.0 mm
- net Net-(D704-Pad1): track 0.00 -> 26.8 mm
- net /VCF/VCF CV Ins/Freq_In: track 0.00 -> 25.6 mm, vias 0 -> 1
- net Net-(R708-Pad1): track 0.00 -> 23.1 mm
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
Commit message: VCF layout done, vca capture
Routing:
- net /+9V: track 803.5 -> 1075.7 mm, vias 30 -> 40
- net /+4.5V: track 894.4 -> 901.1 mm
- net /VCF/VCA_VC1: track 164.7 -> 166.6 mm
- net Net-(R615-Pad2): track 187.8 -> 186.0 mm
- net /VCF/UBP_Vert: track 13.2 -> 11.9 mm
- net /GND: track 57.7 -> 59.0 mm, vias 52 -> 53
- net /VCF/LP: track 110.7 -> 111.7 mm
- net Net-(R704-Pad1): track 21.5 -> 22.3 mm

Commit message: CV VCA & Mixer, Audio VCA schem capture
Parts:
- added C202: 100n, Capacitor_SMD:C_0603_1608Metric_Pad1.08x0.95mm_HandSolder, F.Cu at (38.6, 199.7)
- added C203: 100n, Capacitor_SMD:C_0603_1608Metric_Pad1.08x0.95mm_HandSolder, F.Cu at (62.7, 226.4)
- added C204: 100n, Capacitor_SMD:C_0603_1608Metric_Pad1.08x0.95mm_HandSolder, F.Cu at (-43.4, 210.1)
- added C205: 100p, Capacitor_SMD:C_0603_1608Metric_Pad1.08x0.95mm_HandSolder, F.Cu at (-43.4, 212.6)
- added C206: 100n, Capacitor_SMD:C_0603_1608Metric_Pad1.08x0.95mm_HandSolder, F.Cu at (70.8, 199.5)
- added C207: 100n, Capacitor_SMD:C_0603_1608Metric_Pad1.08x0.95mm_HandSolder, F.Cu at (77.7, 224.7)
- added C208: 100n, Capacitor_SMD:C_0603_1608Metric_Pad1.08x0.95mm_HandSolder, F.Cu at (-36.4, 220.1)
- added C209: 100n, Capacitor_SMD:C_0603_1608Metric_Pad1.08x0.95mm_HandSolder, F.Cu at (69.3, 209.4)
- added C901: 100p, Capacitor_SMD:C_0603_1608Metric_Pad1.08x0.95mm_HandSolder, F.Cu at (540.5, -14.6)
- added C902: 10p, Capacitor_SMD:C_0603_1608Metric_Pad1.08x0.95mm_HandSolder, F.Cu at (552.7, -22.2)
- added C903: 100p, Capacitor_SMD:C_0603_1608Metric_Pad1.08x0.95mm_HandSolder, F.Cu at (563.1, -29.7)
- added C904: 10p, Capacitor_SMD:C_0603_1608Metric_Pad1.08x0.95mm_HandSolder, F.Cu at (544.2, -19.6)
- added C905: 10p, Capacitor_SMD:C_0603_1608Metric_Pad1.08x0.95mm_HandSolder, F.Cu at (554.4, -32.2)
- added C906: 10p, Capacitor_SMD:C_0603_1608Metric_Pad1.08x0.95mm_HandSolder, F.Cu at (548.3, -22.2)
- added C907: 100n, Capacitor_SMD:C_0603_1608Metric_Pad1.08x0.95mm_HandSolder, F.Cu at (531.8, -12.4)
- added C908: 100n, Capacitor_SMD:C_0603_1608Metric_Pad1.08x0.95mm_HandSolder, F.Cu at (540.3, -17.1)
- added C909: 100n, Capacitor_SMD:C_0603_1608Metric_Pad1.08x0.95mm_HandSolder, F.Cu at (563.1, -32.2)
- added D1001: D_TVS, Diode_SMD:D_SOD-323_HandSoldering, F.Cu at (566.3, -58.3)
- added D1002: D_TVS, Diode_SMD:D_SOD-323_HandSoldering, F.Cu at (561.2, -51.1)
- added D1003: D_TVS, Diode_SMD:D_SOD-323_HandSoldering, F.Cu at (576.5, -68.4)
- added D1004: D_TVS, Diode_SMD:D_SOD-323_HandSoldering, F.Cu at (566.3, -61.2)
- added D1005: D_TVS, Diode_SMD:D_SOD-323_HandSoldering, F.Cu at (535.8, -40.9)
- added D1006: D_TVS, Diode_SMD:D_SOD-323_HandSoldering, F.Cu at (540.9, -40.9)
- added D1007: D_TVS, Diode_SMD:D_SOD-323_HandSoldering, F.Cu at (556.2, -51.1)
- added D1008: D_TVS, Diode_SMD:D_SOD-323_HandSoldering, F.Cu at (556.2, -48.1)
- added D1009: D_TVS, Diode_SMD:D_SOD-323_HandSoldering, F.Cu at (576.5, -71.4)
- added D1010: D_TVS, Diode_SMD:D_SOD-323_HandSoldering, F.Cu at (530.8, -40.9)
- added D1011: D_TVS, Diode_SMD:D_SOD-323_HandSoldering, F.Cu at (525.7, -40.9)
- added D1012: D_TVS, Diode_SMD:D_SOD-323_HandSoldering, F.Cu at (545.9, -40.9)
- added D1101: D_TVS, Diode_SMD:D_SOD-323_HandSoldering, F.Cu at (28.6, 206.3)
- added D1102: D_TVS, Diode_SMD:D_SOD-323_HandSoldering, F.Cu at (52.8, 200.2)
- added D1103: D_TVS, Diode_SMD:D_SOD-323_HandSoldering, F.Cu at (77.2, 200.5)
- added D1104: D_TVS, Diode_SMD:D_SOD-323_HandSoldering, F.Cu at (101.8, 206.3)
- added D1105: D_TVS, Diode_SMD:D_SOD-323_HandSoldering, F.Cu at (52.8, 226.9)
- added D1106: D_TVS, Diode_SMD:D_SOD-323_HandSoldering, F.Cu at (101.8, 218.3)
- added H1001: VCA1_In, MountingHole:MountingHole_4.3mm_M4_Pad_TopBottom, F.Cu at (548.6, -47.5)
- added H1002: VCA1_CV_In, MountingHole:MountingHole_4.3mm_M4_Pad_TopBottom, F.Cu at (528.3, -47.5)
- added H1003: VCA2_In, MountingHole:MountingHole_4.3mm_M4_Pad_TopBottom, F.Cu at (538.4, -67.8)
- added H1004: VCA2_CV_In, MountingHole:MountingHole_4.3mm_M4_Pad_TopBottom, F.Cu at (528.3, -57.6)
- added H1005: VCA1_Out, MountingHole:MountingHole_4.3mm_M4_Pad_TopBottom, F.Cu at (538.4, -47.5)
- added H1006: VCA2_Out, MountingHole:MountingHole_4.3mm_M4_Pad_TopBottom, F.Cu at (558.7, -67.8)
- added H1007: Mixer1_In1, MountingHole:MountingHole_4.3mm_M4_Pad_TopBottom, F.Cu at (568.9, -67.8)
- added H1008: Mixer1_In2, MountingHole:MountingHole_4.3mm_M4_Pad_TopBottom, F.Cu at (548.6, -67.8)
- added H1009: Mixer2_In1, MountingHole:MountingHole_4.3mm_M4_Pad_TopBottom, F.Cu at (548.6, -57.6)
- added H1010: Mixer2_In2, MountingHole:MountingHole_4.3mm_M4_Pad_TopBottom, F.Cu at (528.3, -67.8)
- added H1011: Mixer1_Out, MountingHole:MountingHole_4.3mm_M4_Pad_TopBottom, F.Cu at (558.7, -57.6)
- added H1012: Mixer2_Out, MountingHole:MountingHole_4.3mm_M4_Pad_TopBottom, F.Cu at (538.4, -57.6)
- added H1101: VCA1_In, MountingHole:MountingHole_4.3mm_M4_Pad_TopBottom, B.Cu at (35.5, 207.6)
- added H1102: VCA1_CV_In, MountingHole:MountingHole_4.3mm_M4_Pad_TopBottom, B.Cu at (52.8, 207.6)
- added H1103: VCA2_In, MountingHole:MountingHole_4.3mm_M4_Pad_TopBottom, B.Cu at (77.0, 207.6)
- added H1104: VCA2_CV_In, MountingHole:MountingHole_4.3mm_M4_Pad_TopBottom, B.Cu at (94.4, 207.6)
- added H1105: VCA1_Out, MountingHole:MountingHole_4.3mm_M4_Pad_TopBottom, B.Cu at (52.8, 219.6)
- added H1106: VCA2_Out, MountingHole:MountingHole_4.3mm_M4_Pad_TopBottom, B.Cu at (94.4, 219.6)
- added Q202: Q_PNP_BEC, Package_TO_SOT_SMD:SOT-23_Handsoldering, F.Cu at (-48.4, 218.7)
- added Q901: Q_PNP_BEC, Package_TO_SOT_SMD:SOT-23_Handsoldering, F.Cu at (526.4, -12.1)
- added Q902: Q_PNP_BEC, Package_TO_SOT_SMD:SOT-23_Handsoldering, F.Cu at (534.9, -16.0)
- added R213: 200K, Resistor_SMD:R_0603_1608Metric_Pad0.98x0.95mm_HandSolder, F.Cu at (41.6, 199.7)
- added R214: 200K, Resistor_SMD:R_0603_1608Metric_Pad0.98x0.95mm_HandSolder, F.Cu at (59.9, 226.4)
- added R215: 1M, Resistor_SMD:R_0603_1608Metric_Pad0.98x0.95mm_HandSolder, F.Cu at (-34.3, 217.6)
- added R216: 100K, Resistor_SMD:R_0603_1608Metric_Pad0.98x0.95mm_HandSolder, F.Cu at (-43.0, 217.6)
- added R217: 100K, Resistor_SMD:R_0603_1608Metric_Pad0.98x0.95mm_HandSolder, F.Cu at (-34.7, 212.6)
- added R218: 200K, Resistor_SMD:R_0603_1608Metric_Pad0.98x0.95mm_HandSolder, F.Cu at (-45.1, 222.2)
- added R219: 10K, Resistor_SMD:R_0603_1608Metric_Pad0.98x0.95mm_HandSolder, F.Cu at (-40.8, 222.7)
- added R220: 1K, Resistor_SMD:R_0603_1608Metric_Pad0.98x0.95mm_HandSolder, F.Cu at (-34.7, 210.1)
- added R221: 680, Resistor_SMD:R_0603_1608Metric_Pad0.98x0.95mm_HandSolder, F.Cu at (-43.0, 215.1)
- added R222: 30K, Resistor_SMD:R_0603_1608Metric_Pad0.98x0.95mm_HandSolder, F.Cu at (-38.7, 215.1)
- added R223: 5K, Resistor_SMD:R_0603_1608Metric_Pad0.98x0.95mm_HandSolder, F.Cu at (-34.3, 215.1)
- added R224: 200K, Resistor_SMD:R_0603_1608Metric_Pad0.98x0.95mm_HandSolder, F.Cu at (-39.1, 210.1)
- added R901: 100K, Resistor_SMD:R_0603_1608Metric_Pad0.98x0.95mm_HandSolder, F.Cu at (558.7, -32.2)
- added R902: 100K, Resistor_SMD:R_0603_1608Metric_Pad0.98x0.95mm_HandSolder, F.Cu at (557.0, -27.2)
- added R903: 100K, Resistor_SMD:R_0603_1608Metric_Pad0.98x0.95mm_HandSolder, F.Cu at (558.7, -34.7)
- added R904: 10K, Resistor_SMD:R_0603_1608Metric_Pad0.98x0.95mm_HandSolder, F.Cu at (557.0, -22.2)
- added R905: 30K, Resistor_SMD:R_0603_1608Metric_Pad0.98x0.95mm_HandSolder, F.Cu at (567.4, -32.2)
- added R906: 1K, Resistor_SMD:R_0603_1608Metric_Pad0.98x0.95mm_HandSolder, F.Cu at (558.7, -29.7)
- added R907: 8.2K, Resistor_SMD:R_0603_1608Metric_Pad0.98x0.95mm_HandSolder, F.Cu at (548.3, -24.7)
- added R908: 680, Resistor_SMD:R_0603_1608Metric_Pad0.98x0.95mm_HandSolder, F.Cu at (548.3, -27.2)
- added R909: 75K, Resistor_SMD:R_0603_1608Metric_Pad0.98x0.95mm_HandSolder, F.Cu at (549.0, -17.1)
- added R910: 100K, Resistor_SMD:R_0603_1608Metric_Pad0.98x0.95mm_HandSolder, F.Cu at (552.7, -27.2)
- added R911: 100K, Resistor_SMD:R_0603_1608Metric_Pad0.98x0.95mm_HandSolder, F.Cu at (553.3, -17.1)
- added R912: 10K, Resistor_SMD:R_0603_1608Metric_Pad0.98x0.95mm_HandSolder, F.Cu at (536.2, -12.4)
- added R913: 1K, Resistor_SMD:R_0603_1608Metric_Pad0.98x0.95mm_HandSolder, F.Cu at (544.9, -14.6)
- added R914: 1K, Resistor_SMD:R_0603_1608Metric_Pad0.98x0.95mm_HandSolder, F.Cu at (557.0, -24.7)
- added R915: 100K, Resistor_SMD:R_0603_1608Metric_Pad0.98x0.95mm_HandSolder, F.Cu at (554.4, -34.7)
- added R916: 680, Resistor_SMD:R_0603_1608Metric_Pad0.98x0.95mm_HandSolder, F.Cu at (557.3, -19.7)
- added R917: 30K, Resistor_SMD:R_0603_1608Metric_Pad0.98x0.95mm_HandSolder, F.Cu at (544.9, -12.1)
- added R918: 8.2K, Resistor_SMD:R_0603_1608Metric_Pad0.98x0.95mm_HandSolder, F.Cu at (548.6, -19.7)
- added R919: 100K, Resistor_SMD:R_0603_1608Metric_Pad0.98x0.95mm_HandSolder, F.Cu at (567.4, -34.7)
- added R920: 100K, Resistor_SMD:R_0603_1608Metric_Pad0.98x0.95mm_HandSolder, F.Cu at (540.5, -12.1)
- added R921: 100K, Resistor_SMD:R_0603_1608Metric_Pad0.98x0.95mm_HandSolder, F.Cu at (544.6, -17.1)
- added R922: 100K, Resistor_SMD:R_0603_1608Metric_Pad0.98x0.95mm_HandSolder, F.Cu at (554.4, -29.7)
- added R923: 100K, Resistor_SMD:R_0603_1608Metric_Pad0.98x0.95mm_HandSolder, F.Cu at (563.1, -34.7)
- added R924: 100K, Resistor_SMD:R_0603_1608Metric_Pad0.98x0.95mm_HandSolder, F.Cu at (552.9, -19.7)
- added R925: 1K, Resistor_SMD:R_0603_1608Metric_Pad0.98x0.95mm_HandSolder, F.Cu at (552.7, -24.7)
- added R926: 1K, Resistor_SMD:R_0603_1608Metric_Pad0.98x0.95mm_HandSolder, F.Cu at (549.2, -14.6)
- added R927: 75K, Resistor_SMD:R_0603_1608Metric_Pad0.98x0.95mm_HandSolder, F.Cu at (561.4, -27.2)
- added R928: 1K, Resistor_SMD:R_0603_1608Metric_Pad0.98x0.95mm_HandSolder, F.Cu at (539.9, -19.6)
- added RV204: 100K, Potentiometer_SMD:Potentiometer_Bourns_3314J_Vertical, F.Cu at (-63.8, 221.3)
- added RV901: 100K, Potentiometer_SMD:Potentiometer_Bourns_3314J_Vertical, F.Cu at (543.1, -32.2)
- added RV902: 1K, Potentiometer_SMD:Potentiometer_Bourns_3314J_Vertical, F.Cu at (549.2, -32.2)
- added RV903: 100K, Potentiometer_SMD:Potentiometer_Bourns_3314J_Vertical, F.Cu at (543.1, -24.7)
- added RV904: 1K, Potentiometer_SMD:Potentiometer_Bourns_3314J_Vertical, F.Cu at (534.7, -22.0)
- added U901: MCP6004, Package_SO:SOIC-14_3.9x8.7mm_P1.27mm, F.Cu at (535.9, -30.9)
- added U902: MCP6004, Package_SO:SOIC-14_3.9x8.7mm_P1.27mm, F.Cu at (527.4, -19.4)
- added U903: LM13700, Package_SO:SOIC-16_3.9x9.9mm_P1.27mm, F.Cu at (527.4, -30.3)
- C201: value 470p -> 100p
- R212: value 20K -> 1M
- RV201: value 100K multiturn -> 100K
- U202: value MCP6004 -> MCP6002; footprint Package_SO:SOIC-14_3.9x8.7mm_P1.27mm -> Package_SO:SOIC-8_3.9x4.9mm_P1.27mm
- U203: value MCP6004 -> TL072; footprint Package_SO:SOIC-14_3.9x8.7mm_P1.27mm -> Package_SO:SOIC-8_3.9x4.9mm_P1.27mm
- moved C201 676.4 mm to (-32.8, 250.4)
- moved R208 676.4 mm to (-20.7, 240.8)
- moved R210 676.4 mm to (-20.7, 235.8)
- moved R211 676.4 mm to (-24.1, 245.8)
- moved RV201 606.2 mm to (41.9, 219.8), turned to 90 degrees
- moved R212 604.6 mm to (35.5, 199.7), turned to 90 degrees
- moved R209 595.5 mm to (39.8, 213.7), turned to -90 degrees
- moved Q201 594.1 mm to (44.9, 213.7), turned to 180 degrees
- moved R202 594.0 mm to (64.4, 217.5)
- moved R205 590.6 mm to (58.1, 212.2), turned to -90 degrees
- moved R201 590.2 mm to (59.6, 206.6), turned to -90 degrees
- moved R204 589.6 mm to (45.9, 208.5), turned to -90 degrees
- moved R207 582.0 mm to (60.1, 217.5), turned to 180 degrees
- moved RV202 581.2 mm to (62.7, 221.3), turned to 90 degrees
- moved R206 580.2 mm to (65.7, 226.4), turned to 90 degrees
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Connections:
- net /2xAttenuverters1/VCF_1_In renamed /2xAttenuverters1/2xAudio VCA_1_In
- net /2xAttenuverters1/VCF_1_Out renamed /2xAttenuverters1/2xAudio VCA_1_Out
- net /2xAttenuverters1/VCF_2_In renamed /2xAttenuverters1/2xAudio VCA_2_In
- net /2xAttenuverters1/VCF_2_Out renamed /2xAttenuverters1/2xAudio VCA_2_Out
- net /2xAttenuverters2/VCF_1_In renamed /2xAttenuverters2/2xAudio VCA_1_In
- net /2xAttenuverters2/VCF_1_Out renamed /2xAttenuverters2/2xAudio VCA_1_Out
- net /2xAttenuverters2/VCF_2_In renamed /2xAttenuverters2/2xAudio VCA_2_In
- net /2xAttenuverters2/VCF_2_Out renamed /2xAttenuverters2/2xAudio VCA_2_Out
- net /2xAttenuverters3/VCF_1_In renamed /2xAttenuverters3/2xAudio VCA_1_In
- net /2xAttenuverters3/VCF_1_Out renamed /2xAttenuverters3/2xAudio VCA_1_Out
- net /2xAttenuverters3/VCF_2_In renamed /2xAttenuverters3/2xAudio VCA_2_In
- net /2xAttenuverters3/VCF_2_Out renamed /2xAttenuverters3/2xAudio VCA_2_Out
- R201 pad 1: /VCA-LM13700/A1_IN -> Net-(R201-Pad1)
- R202 pad 1: /VCA-LM13700/+9V -> /+9V
- R204 pad 1: /VCA-LM13700/CV1_IN -> /2xAudio VCA/VCA1_CV
- R206 pad 2: /VCA-LM13700/+4.5V -> /+4.5V
- R207 pad 1: /VCA-LM13700/Iabc1 -> /2xAudio VCA/VCA1_Iabc
- R208 pad 2: /VCA-LM13700/GND -> /GND
- R209 pad 2: /VCA-LM13700/+4.5V -> /+4.5V
- R210 pad 1: unconnected-(R210-Pad1) -> Net-(R210-Pad1)
- R211 pad 1: /VCA-LM13700/+9V -> /+9V
- R212 pad 1: Net-(R212-Pad1) -> /2xAudio VCA/VCA1_In
- R212 pad 2: Net-(R212-Pad2) -> /GND
- RV201 pad 1: /VCA-LM13700/+9V -> /+9V
- RV201 pad 3: /VCA-LM13700/GND -> /GND
- RV202 pad 2: /VCA-LM13700/+4.5V -> /+4.5V
- RV203 pad 2: /VCA-LM13700/+4.5V -> /+4.5V
- U201 pad 1: unconnected-(U201-Pad1) -> /2xAudio VCA/VCA1_Iabc
- U201 pad 10: Net-(R206-Pad1) -> Net-(R222-Pad1)
- U201 pad 11: unconnected-(U201-Pad11) -> /+9V
- U201 pad 12: Net-(R206-Pad1) -> Net-(R222-Pad1)
- U201 pad 13: Net-(RV202-Pad3) -> Net-(RV203-Pad3)
- U201 pad 14: Net-(R201-Pad2) -> Net-(R210-Pad2)
- U201 pad 15: Net-(R202-Pad2) -> Net-(R211-Pad2)
- U201 pad 16: /VCA-LM13700/Iabc1 -> /2xAudio VCA/VCA2_Iabc
- U201 pad 2: Net-(R211-Pad2) -> Net-(R202-Pad2)
- U201 pad 3: Net-(R210-Pad2) -> Net-(R201-Pad2)
- U201 pad 4: Net-(RV203-Pad3) -> Net-(RV202-Pad3)
- U201 pad 5: Net-(R212-Pad1) -> Net-(R206-Pad1)
- U201 pad 6: unconnected-(U201-Pad6) -> /GND
- U201 pad 7: unconnected-(U201-Pad7) -> Net-(R206-Pad1)
- U201 pad 8: unconnected-(U201-Pad8) -> Net-(R208-Pad1)
- U201 pad 9: Net-(R208-Pad1) -> Net-(C208-Pad1)
- U202 pad 3: /VCA-LM13700/+4.5V -> /+4.5V
- U202 pad 4: (no net) -> /GND
- U202 pad 5: (no net) -> /+4.5V
- U202 pad 6: (no net) -> Net-(C205-Pad1)
- U202 pad 7: (no net) -> Net-(Q202-Pad1)
- U202 pad 8: (no net) -> /+9V
- U203 pad 1: Net-(R212-Pad2) -> Net-(R201-Pad1)
- U203 pad 2: Net-(R212-Pad1) -> Net-(R201-Pad1)
- U203 pad 3: /VCA-LM13700/+4.5V -> Net-(C202-Pad2)
- U203 pad 4: (no net) -> /GND
- U203 pad 5: (no net) -> Net-(C204-Pad2)
- U203 pad 6: (no net) -> Net-(R210-Pad1)
- U203 pad 7: (no net) -> Net-(R210-Pad1)
- U203 pad 8: (no net) -> /+9V
