File: audio-jacks.kicad_sch (KiCad schematic)
At the start: 58 parts

Commit message: Mixer redesign wip
Parts:
- added C2909, C2910, C2911, C2912: 100n, Capacitor_SMD:C_0603_1608Metric_Pad1.08x0.95mm_HandSolder, symbol Device:C
- gave numbers to parts that had none: 58
Connections:
- net +9V: now also C2909.1, C2910.1, C2911.1, C2912.1
- net GND: now also C2909.2, C2910.2, C2911.2, C2912.2

Commit message: Add JLC parts numbers
Parts:
- C2901, C2905: LCSC (none) -> C38141; Role (none) -> audio-coupling
- C2902, C2903, C2904, C2906, C2907, C2908: LCSC (none) -> C651004; Role (none) -> audio-coupling
- C2909, C2910, C2911, C2912: LCSC (none) -> C497032; Role (none) -> ic-bypass
- D2901, D2902, D2903, D2904, D2905, D2906, D2907, D2908, D2909, D2910, D2911, D2912: LCSC (none) -> C20936
- Q2901, Q2903: LCSC (none) -> C891687
- Q2902, Q2904: value 3904 -> 3904 BEC; LCSC (none) -> C20526
- R2901, R2902, R2903, R2909, R2910, R2911: LCSC (none) -> C234360
- R2904, R2907, R2908, R2912, R2915, R2916: LCSC (none) -> C203392
- R2905, R2906, R2913, R2914: LCSC (none) -> C144661
