File: audio-vca-io.kicad_sch (KiCad schematic)
At the start: 12 parts

Commit message: Add JLC parts numbers
Parts:
- D1101, D1102, D1103, D1104, D1105, D1106: LCSC (none) -> C20936
Changed lines of the file:
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@@
+      (effects (font (size 1.27 1.27)) hide)
+    )
+    (property "LCSC" "C20936" (id 4) (at 33.02 67.945 0)
       (effects (font (size 1.27 1.27)) hide)
     )
@@
       (effects (font (size 1.27 1.27)) hide)
     )
+    (property "LCSC" "C20936" (id 4) (at 33.02 139.065 0)
+      (effects (font (size 1.27 1.27)) hide)
+    )
     (pin "1")
     (pin "2")
@@
     )
     (property "Datasheet" "~" (id 3) (at 33.02 106.045 0)
+      (effects (font (size 1.27 1.27)) hide)
+    )
+    (property "LCSC" "C20936" (id 4) (at 33.02 106.045 0)
       (effects (font (size 1.27 1.27)) hide)
     )
@@
       (effects (font (size 1.27 1.27)) hide)
     )
+    (property "LCSC" "C20936" (id 4) (at 72.39 32.385 0)
+      (effects (font (size 1.27 1.27)) hide)
+    )
     (pin "1")
     (pin "2")
@@
       (effects (font (size 1.27 1.27)) hide)
     )
+    (property "LCSC" "C20936" (id 4) (at 33.02 32.385 0)
+      (effects (font (size 1.27 1.27)) hide)
+    )
     (pin "1")
     (pin "2")
@@
       (effects (font (size 1.27 1.27)) hide)
     )
+    (property "LCSC" "C20936" (id 4) (at 72.39 106.045 0)
+      (effects (font (size 1.27 1.27)) hide)
+    )
