File: relay-switch.kicad_sch (KiCad schematic)
At the start: 60 parts, among them U2401 TL072, U2402 4013

Commit message: Relay switch layout done
Parts:
- H2401: renamed from H?; value In1 -> Switch1_Trig
- H2402: renamed from H?; value In1 -> Switch2_Trig
- H2403: renamed from H?; value In1 -> Switch1_A
- H2404: renamed from H?; value In1 -> Switch2_A
- H2405: renamed from H?; value In1 -> Switch1_B
- H2406: renamed from H?; value In1 -> Switch2_B
- H2407: renamed from H?; value In1 -> Switch1_AorB
- H2408: renamed from H?; value In1 -> Switch2_AorB
- H2409: renamed from H?; value In1 -> Switch1_C
- H2410: renamed from H?; value In1 -> Switch2_C
- H2411: renamed from H?; value In1 -> Switch1_D
- H2412: renamed from H?; value In1 -> Switch2_D
- H2413: renamed from H?; value In1 -> Switch1_CorD
- H2414: renamed from H?; value In1 -> Switch2_CorD
- gave numbers to parts that had none: 14
Connections:
- net +9V: now also C2403.1, C2404.1, U2401.8 (V+), U2402.14 (VDD)
- net GND: now also C2403.2, C2404.2, U2401.4 (V-), U2402.7 (VSS)

Commit message: Add JLC parts numbers
Parts:
- C2401, C2402: LCSC (none) -> C519438; Role (none) -> cv-filter
- C2403, C2404: LCSC (none) -> C497032; Role (none) -> ic-bypass
- D2405, D2406, D2407, D2408: LCSC (none) -> C122841
- D2409, D2410, D2411, D2412, D2413, D2414, D2415, D2416, D2417, D2418, D2419, D2420, D2421, D2422: LCSC (none) -> C20936
- R2401, R2402, R2411, R2412: LCSC (none) -> C2907002
- R2403, R2404, R2405, R2406, R2407, R2408, R2409, R2410: LCSC (none) -> C14675
- R2413, R2414, R2415, R2416: LCSC (none) -> C98220
- RL2401, RL2402: LCSC (none) -> C2961043
- U2401: LCSC (none) -> C67473
- U2402: LCSC (none) -> C194333
