File: slew-limiter.kicad_sch (KiCad schematic)
At the start: 18 parts, among them SW2701 SW_DIP_x02, U2701 TL972

Commit message: Add JLC parts numbers
Parts:
- C2701: LCSC (none) -> C511013; Role (none) -> cv-filter
- C2702: LCSC (none) -> C2798037; Role (none) -> cv-filter
- C2703: LCSC (none) -> C140402; Role (none) -> cv-filter
- C2704: LCSC (none) -> C497032; Role (none) -> ic-bypass
- D2701, D2702: LCSC (none) -> C20936
- D2703, D2704: LCSC (none) -> C2128
- R2701: LCSC (none) -> C14675
- R2702, R2704: LCSC (none) -> C2907002
- R2703: LCSC (none) -> C98220
- U2701: LCSC (none) -> C46127
Changed lines of the file:
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@@
+      (effects (font (size 1.27 1.27)) hide)
+    )
+    (property "LCSC" "C2128" (id 4) (at 96.52 41.91 0)
       (effects (font (size 1.27 1.27)) hide)
     )
@@
       (effects (font (size 1.27 1.27)) hide)
     )
-    (property "LCSC" "" (id 4) (at 113.03 59.69 0)
+    (property "LCSC" "C511013" (id 4) (at 113.03 59.69 0)
+      (effects (font (size 1.27 1.27)) hide)
+    )
+    (property "Role" "cv-filter" (id 5) (at 113.03 59.69 0)
       (effects (font (size 1.27 1.27)) hide)
     )
@@
     )
     (property "Datasheet" "http://ww1.microchip.com/downloads/en/DeviceDoc/21733j.pdf" (id 3) (at 144.78 54.61 0)
+      (effects (font (size 1.27 1.27)) hide)
+    )
+    (property "LCSC" "C46127" (id 4) (at 144.78 54.61 0)
       (effects (font (size 1.27 1.27)) hide)
     )
@@
       (effects (font (size 1.27 1.27)) hide)
     )
-    (property "LCSC" "" (id 4) (at 118.745 78.74 0)
+    (property "LCSC" "C2798037" (id 4) (at 118.745 78.74 0)
+      (effects (font (size 1.27 1.27)) hide)
+    )
+    (property "Role" "cv-filter" (id 5) (at 118.745 78.74 0)
       (effects (font (size 1.27 1.27)) hide)
     )
@@
       (effects (font (size 1.27 1.27)) hide)
     )
+    (property "LCSC" "C2907002" (id 4) (at 60.96 50.8 0)
+      (effects (font (size 1.27 1.27)) hide)
+    )
     (pin "1")
     (pin "2")
@@
       (effects (font (size 1.27 1.27)) hide)
     )
+    (property "LCSC" "C2907002" (id 4) (at 160.02 54.61 0)
+      (effects (font (size 1.27 1.27)) hide)
+    )
     (pin "1")
     (pin "2")
@@
       (effects (font (size 1.27 1.27)) hide)
     )
-    (property "LCSC" "" (id 4) (at 132.715 78.74 0)
+    (property "LCSC" "C140402" (id 4) (at 132.715 78.74 0)
+      (effects (font (size 1.27 1.27)) hide)
+    )
+    (property "Role" "cv-filter" (id 5) (at 132.715 78.74 0)
       (effects (font (size 1.27 1.27)) hide)
     )
@@
       (effects (font (size 1.27 1.27)) hide)
     )
+    (property "LCSC" "C2128" (id 4) (at 96.52 57.15 0)
+      (effects (font (size 1.27 1.27)) hide)
+    )
     (pin "1")
     (pin "2")
@@
     )
     (property "Datasheet" "http://ww1.microchip.com/downloads/en/DeviceDoc/21733j.pdf" (id 3) (at 45.72 50.8 0)
+      (effects (font (size 1.27 1.27)) hide)
+    )
+    (property "LCSC" "C46127" (id 4) (at 45.72 50.8 0)
       (effects (font (size 1.27 1.27)) hide)
     )
@@
       (effects (font (size 1.27 1.27)) hide)
     )
+    (property "LCSC" "C20936" (id 4) (at 35.56 125.73 0)
+      (effects (font (size 1.27 1.27)) hide)
+    )
     (pin "1")
     (pin "2")
@@
       (effects (font (size 1.27 1.27)) hide)
     )
+    (property "LCSC" "C14675" (id 4) (at 33.02 57.15 0)
+      (effects (font (size 1.27 1.27)) hide)
+    )
     (pin "1")
     (pin "2")
@@
       (effects (font (size 1.27 1.27)) hide)
     )
+    (property "LCSC" "C98220" (id 4) (at 96.52 26.67 0)
+      (effects (font (size 1.27 1.27)) hide)
+    )
     (pin "1")
     (pin "2")
@@
       (effects (font (size 1.27 1.27)) hide)
     )
+    (property "LCSC" "C497032" (id 4) (at 251.46 49.53 0)
+      (effects (font (size 1.27 1.27)) hide)
+    )
+    (property "Role" "ic-bypass" (id 5) (at 251.46 49.53 0)
+      (effects (font (size 1.27 1.27)) hide)
+    )
     (pin "1")
     (pin "2")
@@
       (effects (font (size 1.27 1.27)) hide)
     )
+    (property "LCSC" "C20936" (id 4) (at 69.85 125.73 0)
+      (effects (font (size 1.27 1.27)) hide)
+    )
     (pin "1")
     (pin "2")
@@
       (effects (font (size 1.27 1.27)) hide)
     )
+    (property "LCSC" "C46127" (id 4) (at 265.43 49.53 0)
+      (effects (font (size 1.27 1.27)) hide)
+    )
