File: vc-limiter.kicad_sch (KiCad schematic)
At the start: 27 parts, among them U2601 TL074

Commit message: Add JLC parts numbers
Parts:
- C2601, C2603: LCSC (none) -> C651004; Role (none) -> audio-coupling
- C2602: LCSC (none) -> C781889; Role (none) -> audio-coupling
- C2604: LCSC (none) -> C497032; Role (none) -> ic-bypass
- D2601, D2602: LCSC (none) -> C2128
- D2603, D2604, D2605, D2606: LCSC (none) -> C20936
- R2601: LCSC (none) -> C234360
- R2602, R2612: LCSC (none) -> C203392
- R2603, R2606, R2607: LCSC (none) -> C14675
- R2604, R2609, R2610: LCSC (none) -> C2907011
- R2605, R2611: LCSC (none) -> C2907002
- R2608: LCSC (none) -> C98220
- U2601: LCSC (none) -> C6963
Changed lines of the file:
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@@
+      (effects (font (size 1.27 1.27)) hide)
+    )
+    (property "LCSC" "C2907002" (id 4) (at 134.62 85.09 0)
       (effects (font (size 1.27 1.27)) hide)
     )
@@
     )
     (property "Datasheet" "~" (id 3) (at 93.98 93.98 0)
+      (effects (font (size 1.27 1.27)) hide)
+    )
+    (property "LCSC" "C98220" (id 4) (at 93.98 93.98 0)
       (effects (font (size 1.27 1.27)) hide)
     )
@@
     )
     (property "Datasheet" "~" (id 3) (at 80.01 129.54 0)
+      (effects (font (size 1.27 1.27)) hide)
+    )
+    (property "LCSC" "C14675" (id 4) (at 80.01 129.54 0)
       (effects (font (size 1.27 1.27)) hide)
     )
@@
       (effects (font (size 1.27 1.27)) hide)
     )
+    (property "LCSC" "C651004" (id 4) (at 38.1 90.17 0)
+      (effects (font (size 1.27 1.27)) hide)
+    )
+    (property "Role" "audio-coupling" (id 5) (at 38.1 90.17 0)
+      (effects (font (size 1.27 1.27)) hide)
+    )
     (pin "1")
     (pin "2")
@@
       (effects (font (size 1.27 1.27)) hide)
     )
+    (property "LCSC" "C14675" (id 4) (at 54.61 134.62 0)
+      (effects (font (size 1.27 1.27)) hide)
+    )
     (pin "1")
     (pin "2")
@@
       (effects (font (size 1.27 1.27)) hide)
     )
+    (property "LCSC" "C234360" (id 4) (at 27.94 93.98 0)
+      (effects (font (size 1.27 1.27)) hide)
+    )
     (pin "1")
     (pin "2")
@@
       (effects (font (size 1.27 1.27)) hide)
     )
+    (property "LCSC" "C2907011" (id 4) (at 63.5 138.43 0)
+      (effects (font (size 1.27 1.27)) hide)
+    )
     (pin "1")
     (pin "2")
@@
       (effects (font (size 1.27 1.27)) hide)
     )
+    (property "LCSC" "C20936" (id 4) (at 184.15 69.85 0)
+      (effects (font (size 1.27 1.27)) hide)
+    )
     (pin "1")
     (pin "2")
@@
       (effects (font (size 1.27 1.27)) hide)
     )
+    (property "LCSC" "C2128" (id 4) (at 104.14 99.06 0)
+      (effects (font (size 1.27 1.27)) hide)
+    )
     (pin "1")
     (pin "2")
@@
       (effects (font (size 1.27 1.27)) hide)
     )
+    (property "LCSC" "C20936" (id 4) (at 218.44 69.85 0)
+      (effects (font (size 1.27 1.27)) hide)
+    )
     (pin "1")
     (pin "2")
@@
     )
     (property "Datasheet" "~" (id 3) (at 252.73 36.83 0)
+      (effects (font (size 1.27 1.27)) hide)
+    )
+    (property "LCSC" "C497032" (id 4) (at 252.73 36.83 0)
+      (effects (font (size 1.27 1.27)) hide)
+    )
+    (property "Role" "ic-bypass" (id 5) (at 252.73 36.83 0)
       (effects (font (size 1.27 1.27)) hide)
     )
@@
       (effects (font (size 1.27 1.27)) hide)
     )
+    (property "LCSC" "C14675" (id 4) (at 80.01 38.1 0)
+      (effects (font (size 1.27 1.27)) hide)
+    )
     (pin "1")
     (pin "2")
@@
     )
     (property "Datasheet" "~" (id 3) (at 48.26 93.98 0)
+      (effects (font (size 1.27 1.27)) hide)
+    )
+    (property "LCSC" "C203392" (id 4) (at 48.26 93.98 0)
       (effects (font (size 1.27 1.27)) hide)
     )
@@
       (effects (font (size 1.27 1.27)) hide)
     )
-    (property "LCSC" "" (id 4) (at 87.63 87.63 0)
+    (property "LCSC" "C781889" (id 4) (at 87.63 87.63 0)
+      (effects (font (size 1.27 1.27)) hide)
+    )
+    (property "Role" "audio-coupling" (id 5) (at 87.63 87.63 0)
       (effects (font (size 1.27 1.27)) hide)
     )
@@
       (effects (font (size 1.27 1.27)) hide)
     )
+    (property "LCSC" "C2128" (id 4) (at 104.14 68.58 0)
+      (effects (font (size 1.27 1.27)) hide)
+    )
     (pin "1")
     (pin "2")
@@
       (effects (font (size 1.27 1.27)) hide)
     )
+    (property "LCSC" "C20936" (id 4) (at 184.15 38.1 0)
+      (effects (font (size 1.27 1.27)) hide)
+    )
     (pin "1")
     (pin "2")
@@
     )
     (property "Datasheet" "~" (id 3) (at 218.44 38.1 0)
+      (effects (font (size 1.27 1.27)) hide)
+    )
+    (property "LCSC" "C20936" (id 4) (at 218.44 38.1 0)
       (effects (font (size 1.27 1.27)) hide)
     )
@@
     )
     (property "Datasheet" "http://www.ti.com/lit/ds/symlink/tl071.pdf" (id 3) (at 120.65 90.17 0)
+      (effects (font (size 1.27 1.27)) hide)
+    )
+    (property "LCSC" "C6963" (id 4) (at 119.38 85.09 0)
       (effects (font (size 1.27 1.27)) hide)
     )
@@
       (effects (font (size 1.27 1.27)) hide)
     )
+    (property "LCSC" "C6963" (id 4) (at 96.52 40.64 0)
+      (effects (font (size 1.27 1.27)) hide)
+    )
     (pin "1")
     (pin "2")
@@
       (effects (font (size 1.27 1.27)) hide)
     )
+    (property "LCSC" "C6963" (id 4) (at 96.52 132.08 0)
+      (effects (font (size 1.27 1.27)) hide)
+    )
     (pin "1")
     (pin "2")
@@
       (effects (font (size 1.27 1.27)) hide)
     )
+    (property "LCSC" "C6963" (id 4) (at 266.7 36.83 0)
+      (effects (font (size 1.27 1.27)) hide)
+    )
     (pin "1")
     (pin "2")
@@
       (effects (font (size 1.27 1.27)) hide)
     )
+    (property "LCSC" "C2907011" (id 4) (at 96.52 118.11 0)
+      (effects (font (size 1.27 1.27)) hide)
+    )
     (pin "1")
     (pin "2")
@@
     )
     (property "Datasheet" "http://www.ti.com/lit/ds/symlink/tl071.pdf" (id 3) (at 63.5 92.71 0)
+      (effects (font (size 1.27 1.27)) hide)
+    )
+    (property "LCSC" "C6963" (id 4) (at 62.23 87.63 0)
       (effects (font (size 1.27 1.27)) hide)
     )
@@
       (effects (font (size 1.27 1.27)) hide)
     )
+    (property "LCSC" "C203392" (id 4) (at 152.4 88.9 0)
+      (effects (font (size 1.27 1.27)) hide)
+    )
     (pin "1")
     (pin "2")
@@
       (effects (font (size 1.27 1.27)) hide)
     )
+    (property "LCSC" "C2907002" (id 4) (at 77.47 87.63 0)
+      (effects (font (size 1.27 1.27)) hide)
+    )
     (pin "1")
     (pin "2")
@@
     )
     (property "Datasheet" "~" (id 3) (at 96.52 26.67 0)
+      (effects (font (size 1.27 1.27)) hide)
+    )
+    (property "LCSC" "C2907011" (id 4) (at 96.52 26.67 0)
       (effects (font (size 1.27 1.27)) hide)
     )
@@
       (effects (font (size 1.27 1.27)) hide)
     )
+    (property "LCSC" "C651004" (id 4) (at 144.78 85.09 0)
+      (effects (font (size 1.27 1.27)) hide)
+    )
+    (property "Role" "audio-coupling" (id 5) (at 144.78 85.09 0)
+      (effects (font (size 1.27 1.27)) hide)
+    )
