File: vcf_audio.kicad_sch (KiCad schematic)
At the start: 32 parts

Commit message: VCF schem combed
Parts:
- removed D?: D_TVS, Diode_SMD:D_SOD-323_HandSoldering, symbol Device:D_TVS
- removed H?: Main_Out, MountingHole:MountingHole_4.3mm_M4_Pad_TopBottom, symbol Mechanical:MountingHole_Pad
- removed R? (x4): 100K, symbol Device:R
- added C805: 100n, Capacitor_SMD:C_0603_1608Metric_Pad1.08x0.95mm_HandSolder, symbol Device:C
- added R809, R810, R811, R812, R813, R814, R815, R816: 100K, Resistor_SMD:R_0603_1608Metric_Pad0.98x0.95mm_HandSolder, symbol Device:R
- added RV801, RV802, RV803, RV804: B100K, R0904NB10KL-25KQ:V2_TRIM_R0904NB10KL-25KQ-, symbol R0904NB10KL-25KQ:R_Potentiometer_Shield
- added unit 4 of U801
- added unit 2 of U801
- added unit 4 of U802
- added unit 2 of U802
- added unit 5 of U802
- C801, C802, C803, C804, C806: renamed from C?; footprint (none) -> Capacitor_SMD:C_0603_1608Metric_Pad1.08x0.95mm_HandSolder
- R801, R802, R803, R804, R805, R806, R807, R808: renamed from R?; footprint (none) -> Resistor_SMD:R_0603_1608Metric_Pad0.98x0.95mm_HandSolder
- U801, U802: renamed from U?; footprint (none) -> Package_SO:SOIC-14_3.9x8.7mm_P1.27mm
- gave numbers to parts that had none: 8
Connections:
- net +4.5V: now also RV801.3, RV802.3, RV803.3, RV804.3
- net GND: now also C806.1, U801.11 (V-), C805.1, RV801.0 (ShieldPin), RV802.0 (ShieldPin), RV803.0 (ShieldPin), RV804.0 (ShieldPin), U802.11 (V-)
- net HP_In: now also R809.1, RV801.1
- net LBP_In: now also U802.3 (+), R811.1, RV803.1; no longer U802.10 (+)
- net LP_In: now also U802.10 (+), R812.1, RV804.1; no longer U802.12 (+)
- net UBP_In: now also U801.10 (+), R810.1, RV802.1; no longer U801.5 (+)
- net +9V: now reaches C806.2, U801.4 (V+)
- net +9V: now also C805.2, U802.4 (V+)
- new net: RV804.2, U802.12 (+)
- new net: R812.2, R816.1, U802.13 (-)
- new net: R802.1, U801.8, U801.9 (-)
- new net: R810.2, R814.1, U801.13 (-)
- new net: R804.1, U802.8, U802.9 (-)
- new net: RV801.2, U801.5 (+)
- new net: R803.1, U802.1, U802.2 (-)
- new net: RV802.2, U801.12 (+)
- new net: R811.2, R815.1, U802.6 (-)
- new net: R809.2, R813.1, U801.6 (-)
- new net: RV803.2, U802.5 (+)
- new net HP_Vert: R813.2, U801.7
- new net LBP_Vert: R815.2, U802.7
- new net LP_Vert: R816.2, U802.14
- new net UBP_Vert: R814.2, U801.14
Other:
- moved on the sheet: C802, C803, C804, C806, D801, D802, D803, D804, H802, H803, H804, R802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

Commit message: Start VCF layout
Connections:
- net HP_In: now also U801.12 (+); no longer U801.3 (+)
- net HP_Vert: now also U801.8; no longer U801.7
- net LBP_In: now also U802.12 (+); no longer U802.3 (+)
- net LBP_Vert: now also U802.8; no longer U802.7
- net LP_In: now also U802.3 (+); no longer U802.10 (+)
- net LP_Vert: now also U802.7; no longer U802.14
- net UBP_In: now also U801.3 (+); no longer U801.10 (+)
- net UBP_Vert: now also U801.7; no longer U801.14
- net at RV804.2: now also U802.5 (+); no longer U802.12 (+)
- net at R812.2, R816.1: now also U802.6 (-); no longer U802.13 (-)
- net at R810.2, R814.1: now also U801.6 (-); no longer U801.13 (-)
- net at RV801.2: now also U801.10 (+); no longer U801.5 (+)
- net at RV802.2: now also U801.5 (+); no longer U801.12 (+)
- net at R811.2, R815.1: now also U802.9 (-); no longer U802.6 (-)
- net at R809.2, R813.1: now also U801.9 (-); no longer U801.6 (-)
- net at RV803.2: now also U802.10 (+); no longer U802.5 (+)
- new net: R801.1, U801.13 (-), U801.14
- new net: R802.1, U801.1, U801.2 (-)
- new net: R804.1, U802.1, U802.2 (-)
- new net: R803.1, U802.13 (-), U802.14
Changed lines of the file:
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@@
     (pin "2")
   )
-  (symbol (lib_id "Amplifier_Operational:TL074") (at 52.07 30.48 0) (mirror x) (unit 1)
+  (symbol (lib_id "Amplifier_Operational:TL074") (at 52.07 30.48 0) (mirror x) (unit 4)
     (in_bom yes) (on_board yes) (fields_autoplaced)
     (property "Reference" "U801" (id 0) (at 52.07 20.32 0))
@@
     (pin "1")
   )
-  (symbol (lib_id "Amplifier_Operational:TL074") (at 180.34 138.43 0) (mirror x) (unit 4)
+  (symbol (lib_id "Amplifier_Operational:TL074") (at 180.34 138.43 0) (mirror x) (unit 2)
     (in_bom yes) (on_board yes) (fields_autoplaced)
     (property "Reference" "U802" (id 0) (at 180.34 128.27 0))
@@
     (pin "4")
   )
-  (symbol (lib_id "Amplifier_Operational:TL074") (at 52.07 66.04 0) (mirror x) (unit 3)
+  (symbol (lib_id "Amplifier_Operational:TL074") (at 52.07 66.04 0) (mirror x) (unit 1)
     (in_bom yes) (on_board yes) (fields_autoplaced)
     (property "Reference" "U801" (id 0) (at 52.07 55.88 0))
@@
     (pin "1")
   )
-  (symbol (lib_id "Amplifier_Operational:TL074") (at 52.07 135.89 0) (mirror x) (unit 3)
+  (symbol (lib_id "Amplifier_Operational:TL074") (at 52.07 135.89 0) (mirror x) (unit 1)
     (in_bom yes) (on_board yes) (fields_autoplaced)
     (property "Reference" "U802" (id 0) (at 52.07 125.73 0))
@@
     (pin "2")
   )
-  (symbol (lib_id "Amplifier_Operational:TL074") (at 180.34 68.58 0) (mirror x) (unit 4)
+  (symbol (lib_id "Amplifier_Operational:TL074") (at 180.34 68.58 0) (mirror x) (unit 2)
     (in_bom yes) (on_board yes) (fields_autoplaced)
     (property "Reference" "U801" (id 0) (at 180.34 58.42 0))
@@
     (pin "2")
   )
-  (symbol (lib_id "Amplifier_Operational:TL074") (at 52.07 101.6 0) (mirror x) (unit 1)
+  (symbol (lib_id "Amplifier_Operational:TL074") (at 52.07 101.6 0) (mirror x) (unit 4)
     (in_bom yes) (on_board yes) (fields_autoplaced)
     (property "Reference" "U802" (id 0) (at 52.07 91.44 0))
@@
     (pin "2")
   )
-  (symbol (lib_id "Amplifier_Operational:TL074") (at 180.34 104.14 0) (mirror x) (unit 2)
+  (symbol (lib_id "Amplifier_Operational:TL074") (at 180.34 104.14 0) (mirror x) (unit 3)
     (in_bom yes) (on_board yes) (fields_autoplaced)
     (property "Reference" "U802" (id 0) (at 180.34 93.98 0))
@@
     (pin "4")
   )
-  (symbol (lib_id "Amplifier_Operational:TL074") (at 180.34 33.02 0) (mirror x) (unit 2)
+  (symbol (lib_id "Amplifier_Operational:TL074") (at 180.34 33.02 0) (mirror x) (unit 3)
     (in_bom yes) (on_board yes) (fields_autoplaced)
     (property "Reference" "U801" (id 0) (at 180.34 22.86 0))

Commit message: Increase the size of dc blocking caps
Parts:
- C801, C802, C803, C804: value 100n -> 470n; footprint Capacitor_SMD:C_0603_1608Metric_Pad1.08x0.95mm_HandSolder -> Capacitor_SMD:C_0805_2012Metric_Pad1.18x1.45mm_HandSolder
Changed lines of the file:
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@@
     (pin "4")
+  )
+  (symbol (lib_id "Device:C") (at 76.2 101.6 90) (unit 1)
+    (in_bom yes) (on_board yes) (fields_autoplaced)
+    (property "Reference" "C803" (id 0) (at 76.2 93.98 90))
+    (property "Value" "470n" (id 1) (at 76.2 96.52 90))
+    (property "Footprint" "Capacitor_SMD:C_0805_2012Metric_Pad1.18x1.45mm_HandSolder" (id 2) (at 80.01 100.6348 0)
+      (effects (font (size 1.27 1.27)) hide)
+    )
+    (property "Datasheet" "~" (id 3) (at 76.2 101.6 0)
+      (effects (font (size 1.27 1.27)) hide)
+    )
+    (pin "1")
+    (pin "2")
   )
   (symbol (lib_id "Device:R") (at 180.34 55.88 90) (unit 1)
@@
     (pin "4")
   )
-  (symbol (lib_id "Device:C") (at 76.2 101.6 90) (unit 1)
-    (in_bom yes) (on_board yes) (fields_autoplaced)
-    (property "Reference" "C803" (id 0) (at 76.2 93.98 90))
-    (property "Value" "100n" (id 1) (at 76.2 96.52 90))
-    (property "Footprint" "Capacitor_SMD:C_0603_1608Metric_Pad1.08x0.95mm_HandSolder" (id 2) (at 80.01 100.6348 0)
-      (effects (font (size 1.27 1.27)) hide)
-    )
-    (property "Datasheet" "~" (id 3) (at 76.2 101.6 0)
-      (effects (font (size 1.27 1.27)) hide)
-    )
-    (pin "1")
-    (pin "2")
-  )
   (symbol (lib_id "Device:R") (at 180.34 125.73 90) (unit 1)
     (in_bom yes) (on_board yes) (fields_autoplaced)
@@
     (pin "4")
   )
+  (symbol (lib_id "Device:C") (at 76.2 66.04 90) (unit 1)
+    (in_bom yes) (on_board yes) (fields_autoplaced)
+    (property "Reference" "C802" (id 0) (at 76.2 58.42 90))
+    (property "Value" "470n" (id 1) (at 76.2 60.96 90))
+    (property "Footprint" "Capacitor_SMD:C_0805_2012Metric_Pad1.18x1.45mm_HandSolder" (id 2) (at 80.01 65.0748 0)
+      (effects (font (size 1.27 1.27)) hide)
+    )
+    (property "Datasheet" "~" (id 3) (at 76.2 66.04 0)
+      (effects (font (size 1.27 1.27)) hide)
+    )
+    (pin "1")
+    (pin "2")
+  )
   (symbol (lib_id "Device:D_TVS") (at 110.49 71.12 90) (unit 1)
     (in_bom yes) (on_board yes) (fields_autoplaced)
@@
     (in_bom yes) (on_board yes) (fields_autoplaced)
     (property "Reference" "C804" (id 0) (at 76.2 128.27 90))
-    (property "Value" "100n" (id 1) (at 76.2 130.81 90))
-    (property "Footprint" "Capacitor_SMD:C_0603_1608Metric_Pad1.08x0.95mm_HandSolder" (id 2) (at 80.01 134.9248 0)
+    (property "Value" "470n" (id 1) (at 76.2 130.81 90))
+    (property "Footprint" "Capacitor_SMD:C_0805_2012Metric_Pad1.18x1.45mm_HandSolder" (id 2) (at 80.01 134.9248 0)
       (effects (font (size 1.27 1.27)) hide)
     )
     (property "Datasheet" "~" (id 3) (at 76.2 135.89 0)
-      (effects (font (size 1.27 1.27)) hide)
-    )
-    (pin "1")
-    (pin "2")
-  )
-  (symbol (lib_id "Device:C") (at 76.2 30.48 90) (unit 1)
-    (in_bom yes) (on_board yes) (fields_autoplaced)
-    (property "Reference" "C801" (id 0) (at 76.2 22.86 90))
-    (property "Value" "100n" (id 1) (at 76.2 25.4 90))
-    (property "Footprint" "Capacitor_SMD:C_0603_1608Metric_Pad1.08x0.95mm_HandSolder" (id 2) (at 80.01 29.5148 0)
-      (effects (font (size 1.27 1.27)) hide)
-    )
-    (property "Datasheet" "~" (id 3) (at 76.2 30.48 0)
       (effects (font (size 1.27 1.27)) hide)
     )
@@
     (pin "3")
   )
-  (symbol (lib_id "Device:C") (at 76.2 66.04 90) (unit 1)
-    (in_bom yes) (on_board yes) (fields_autoplaced)
-    (property "Reference" "C802" (id 0) (at 76.2 58.42 90))
-    (property "Value" "100n" (id 1) (at 76.2 60.96 90))
-    (property "Footprint" "Capacitor_SMD:C_0603_1608Metric_Pad1.08x0.95mm_HandSolder" (id 2) (at 80.01 65.0748 0)
-      (effects (font (size 1.27 1.27)) hide)
-    )
-    (property "Datasheet" "~" (id 3) (at 76.2 66.04 0)
-      (effects (font (size 1.27 1.27)) hide)
-    )
+  (symbol (lib_id "Device:C") (at 76.2 30.48 90) (unit 1)
+    (in_bom yes) (on_board yes) (fields_autoplaced)
+    (property "Reference" "C801" (id 0) (at 76.2 22.86 90))
+    (property "Value" "470n" (id 1) (at 76.2 25.4 90))
+    (property "Footprint" "Capacitor_SMD:C_0805_2012Metric_Pad1.18x1.45mm_HandSolder" (id 2) (at 80.01 29.5148 0)
+      (effects (font (size 1.27 1.27)) hide)
+    )
+    (property "Datasheet" "~" (id 3) (at 76.2 30.48 0)
+      (effects (font (size 1.27 1.27)) hide)
+    )

Commit message: Add JLC parts numbers
Parts:
- C801, C802, C803, C804: LCSC (none) -> C651004; Role (none) -> audio-coupling
- C805, C806: LCSC (none) -> C497032; Role (none) -> ic-bypass
- D801, D802, D803, D804: LCSC (none) -> C20936
- R801, R802, R803, R804: LCSC (none) -> C2907002
- R805, R806, R807, R808: LCSC (none) -> C203392
- R809, R810, R811, R812, R813, R814, R815, R816: LCSC (none) -> C14675
- U801, U802: LCSC (none) -> C6963
Changed lines of the file:
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@@
+      (effects (font (size 1.27 1.27)) hide)
+    )
+    (property "LCSC" "C203392" (id 4) (at 82.55 69.85 0)
       (effects (font (size 1.27 1.27)) hide)
     )
@@
     )
     (property "Datasheet" "~" (id 3) (at 82.55 34.29 0)
+      (effects (font (size 1.27 1.27)) hide)
+    )
+    (property "LCSC" "C203392" (id 4) (at 82.55 34.29 0)
       (effects (font (size 1.27 1.27)) hide)
     )
@@
       (effects (font (size 1.27 1.27)) hide)
     )
+    (property "LCSC" "C6963" (id 4) (at 52.07 30.48 0)
+      (effects (font (size 1.27 1.27)) hide)
+    )
     (pin "1")
     (pin "2")
@@
       (effects (font (size 1.27 1.27)) hide)
     )
+    (property "LCSC" "C6963" (id 4) (at 180.34 138.43 0)
+      (effects (font (size 1.27 1.27)) hide)
+    )
     (pin "1")
     (pin "2")
@@
       (effects (font (size 1.27 1.27)) hide)
     )
+    (property "LCSC" "C6963" (id 4) (at 52.07 66.04 0)
+      (effects (font (size 1.27 1.27)) hide)
+    )
     (pin "1")
     (pin "2")
@@
       (effects (font (size 1.27 1.27)) hide)
     )
+    (property "LCSC" "C651004" (id 4) (at 76.2 101.6 0)
+      (effects (font (size 1.27 1.27)) hide)
+    )
+    (property "Role" "audio-coupling" (id 5) (at 76.2 101.6 0)
+      (effects (font (size 1.27 1.27)) hide)
+    )
     (pin "1")
     (pin "2")
@@
       (effects (font (size 1.27 1.27)) hide)
     )
+    (property "LCSC" "C14675" (id 4) (at 180.34 55.88 0)
+      (effects (font (size 1.27 1.27)) hide)
+    )
     (pin "1")
     (pin "2")
@@
       (effects (font (size 1.27 1.27)) hide)
     )
+    (property "LCSC" "C6963" (id 4) (at 52.07 135.89 0)
+      (effects (font (size 1.27 1.27)) hide)
+    )
     (pin "1")
     (pin "2")
@@
       (effects (font (size 1.27 1.27)) hide)
     )
+    (property "LCSC" "C6963" (id 4) (at 269.24 29.21 0)
+      (effects (font (size 1.27 1.27)) hide)
+    )
     (pin "1")
     (pin "2")
@@
     )
     (property "Datasheet" "~" (id 3) (at 110.49 140.97 0)
+      (effects (font (size 1.27 1.27)) hide)
+    )
+    (property "LCSC" "C20936" (id 4) (at 110.49 140.97 0)
       (effects (font (size 1.27 1.27)) hide)
     )
@@
       (effects (font (size 1.27 1.27)) hide)
     )
+    (property "LCSC" "C2907002" (id 4) (at 64.77 135.89 0)
+      (effects (font (size 1.27 1.27)) hide)
+    )
     (pin "1")
     (pin "2")
@@
       (effects (font (size 1.27 1.27)) hide)
     )
+    (property "LCSC" "C2907002" (id 4) (at 64.77 101.6 0)
+      (effects (font (size 1.27 1.27)) hide)
+    )
     (pin "1")
     (pin "2")
@@
     )
     (property "Datasheet" "~" (id 3) (at 82.55 105.41 0)
+      (effects (font (size 1.27 1.27)) hide)
+    )
+    (property "LCSC" "C203392" (id 4) (at 82.55 105.41 0)
       (effects (font (size 1.27 1.27)) hide)
     )
@@
     )
     (property "Datasheet" "http://www.ti.com/lit/ds/symlink/tl071.pdf" (id 3) (at 181.61 73.66 0)
+      (effects (font (size 1.27 1.27)) hide)
+    )
+    (property "LCSC" "C6963" (id 4) (at 180.34 68.58 0)
       (effects (font (size 1.27 1.27)) hide)
     )
@@
       (effects (font (size 1.27 1.27)) hide)
     )
+    (property "LCSC" "C14675" (id 4) (at 180.34 91.44 0)
+      (effects (font (size 1.27 1.27)) hide)
+    )
     (pin "1")
     (pin "2")
@@
     )
     (property "Datasheet" "~" (id 3) (at 255.27 29.21 0)
+      (effects (font (size 1.27 1.27)) hide)
+    )
+    (property "LCSC" "C497032" (id 4) (at 255.27 29.21 0)
+      (effects (font (size 1.27 1.27)) hide)
+    )
+    (property "Role" "ic-bypass" (id 5) (at 255.27 29.21 0)
       (effects (font (size 1.27 1.27)) hide)
     )
@@
       (effects (font (size 1.27 1.27)) hide)
     )
+    (property "LCSC" "C6963" (id 4) (at 52.07 101.6 0)
+      (effects (font (size 1.27 1.27)) hide)
+    )
     (pin "1")
     (pin "2")
@@
       (effects (font (size 1.27 1.27)) hide)
     )
+    (property "LCSC" "C14675" (id 4) (at 180.34 125.73 0)
+      (effects (font (size 1.27 1.27)) hide)
+    )
     (pin "1")
     (pin "2")
@@
       (effects (font (size 1.27 1.27)) hide)
     )
+    (property "LCSC" "C14675" (id 4) (at 165.1 30.48 0)
+      (effects (font (size 1.27 1.27)) hide)
+    )
     (pin "1")
     (pin "2")
@@
       (effects (font (size 1.27 1.27)) hide)
     )
+    (property "LCSC" "C14675" (id 4) (at 165.1 135.89 0)
+      (effects (font (size 1.27 1.27)) hide)
+    )
     (pin "1")
     (pin "2")
@@
     )
     (property "Datasheet" "~" (id 3) (at 110.49 106.68 0)
+      (effects (font (size 1.27 1.27)) hide)
+    )
+    (property "LCSC" "C20936" (id 4) (at 110.49 106.68 0)
       (effects (font (size 1.27 1.27)) hide)
     )
@@
       (effects (font (size 1.27 1.27)) hide)
     )
+    (property "LCSC" "C2907002" (id 4) (at 64.77 66.04 0)
+      (effects (font (size 1.27 1.27)) hide)
+    )
     (pin "1")
     (pin "2")
@@
       (effects (font (size 1.27 1.27)) hide)
     )
+    (property "LCSC" "C14675" (id 4) (at 165.1 66.04 0)
+      (effects (font (size 1.27 1.27)) hide)
+    )
     (pin "1")
     (pin "2")
@@
       (effects (font (size 1.27 1.27)) hide)
     )
+    (property "LCSC" "C2907002" (id 4) (at 64.77 30.48 0)
+      (effects (font (size 1.27 1.27)) hide)
+    )
     (pin "1")
     (pin "2")
@@
       (effects (font (size 1.27 1.27)) hide)
     )
+    (property "LCSC" "C14675" (id 4) (at 180.34 20.32 0)
+      (effects (font (size 1.27 1.27)) hide)
+    )
     (pin "1")
     (pin "2")
@@
     )
     (property "Datasheet" "~" (id 3) (at 110.49 35.56 0)
+      (effects (font (size 1.27 1.27)) hide)
+    )
+    (property "LCSC" "C20936" (id 4) (at 110.49 35.56 0)
       (effects (font (size 1.27 1.27)) hide)
     )
@@
       (effects (font (size 1.27 1.27)) hide)
     )
+    (property "LCSC" "C6963" (id 4) (at 180.34 104.14 0)
+      (effects (font (size 1.27 1.27)) hide)
+    )
     (pin "1")
     (pin "2")
@@
       (effects (font (size 1.27 1.27)) hide)
     )
+    (property "LCSC" "C6963" (id 4) (at 180.34 33.02 0)
+      (effects (font (size 1.27 1.27)) hide)
+    )
     (pin "1")
     (pin "2")
@@
     )
     (property "Datasheet" "http://www.ti.com/lit/ds/symlink/tl071.pdf" (id 3) (at 279.4 24.13 0)
+      (effects (font (size 1.27 1.27)) hide)
+    )
+    (property "LCSC" "C6963" (id 4) (at 278.13 29.21 0)
       (effects (font (size 1.27 1.27)) hide)
     )
@@
       (effects (font (size 1.27 1.27)) hide)
     )
+    (property "LCSC" "C651004" (id 4) (at 76.2 66.04 0)
+      (effects (font (size 1.27 1.27)) hide)
+    )
+    (property "Role" "audio-coupling" (id 5) (at 76.2 66.04 0)
+      (effects (font (size 1.27 1.27)) hide)
+    )
     (pin "1")
     (pin "2")
@@
     )
     (property "Datasheet" "~" (id 3) (at 110.49 71.12 0)
+      (effects (font (size 1.27 1.27)) hide)
+    )
+    (property "LCSC" "C20936" (id 4) (at 110.49 71.12 0)
       (effects (font (size 1.27 1.27)) hide)
     )
@@
       (effects (font (size 1.27 1.27)) hide)
     )
+    (property "LCSC" "C651004" (id 4) (at 76.2 135.89 0)
+      (effects (font (size 1.27 1.27)) hide)
+    )
+    (property "Role" "audio-coupling" (id 5) (at 76.2 135.89 0)
+      (effects (font (size 1.27 1.27)) hide)
+    )
     (pin "1")
     (pin "2")
@@
       (effects (font (size 1.27 1.27)) hide)
     )
+    (property "LCSC" "C497032" (id 4) (at 243.84 29.21 0)
+      (effects (font (size 1.27 1.27)) hide)
+    )
+    (property "Role" "ic-bypass" (id 5) (at 243.84 29.21 0)
+      (effects (font (size 1.27 1.27)) hide)
+    )
     (pin "1")
     (pin "2")
@@
       (effects (font (size 1.27 1.27)) hide)
     )
+    (property "LCSC" "C14675" (id 4) (at 165.1 101.6 0)
+      (effects (font (size 1.27 1.27)) hide)
+    )
     (pin "1")
     (pin "2")
@@
     )
     (property "Datasheet" "~" (id 3) (at 82.55 139.7 0)
+      (effects (font (size 1.27 1.27)) hide)
+    )
+    (property "LCSC" "C203392" (id 4) (at 82.55 139.7 0)
       (effects (font (size 1.27 1.27)) hide)
     )
@@
       (effects (font (size 1.27 1.27)) hide)
     )
+    (property "LCSC" "C651004" (id 4) (at 76.2 30.48 0)
+      (effects (font (size 1.27 1.27)) hide)
+    )
+    (property "Role" "audio-coupling" (id 5) (at 76.2 30.48 0)
+      (effects (font (size 1.27 1.27)) hide)
+    )
